Commit message: Fix mit humanoid model

File: robot-models/mit_humanoid.xacro (robot description, xacro)
@@ -121,5 +121,5 @@
         <link name="${prefix}knee_link">
             <inertial>
-                <mass value="0.35434"/>
+                <mass value="0.35435"/>
                 <origin xyz="0.00528 ${y_sign * -0.0014762} -0.13201"/>
                 <inertia ixx="0.003051" ixy="0.0" ixz="0.0000873"

File: robot-models/mit_humanoid_leg.xacro (robot description, xacro)
@@ -121,5 +121,5 @@
         <link name="${prefix}knee_link">
             <inertial>
-                <mass value="0.35434"/>
+                <mass value="0.35435"/>
                 <origin xyz="0.00528 ${y_sign * 0.0014762} -0.13201"/>
                 <inertia ixx="0.003051" ixy="0.0" ixz="0.0000873"
