Commit message: Ensure dimensions of models match

File: robot-models/double_pendulum.urdf (robot description, URDF)
Before this commit: robot double_pendulum, 3 links, 2 joints
Joints:
- joint joint1: limit (none) -> lower=-3.14 upper=3.14 effort=30 velocity=1.0; type continuous -> revolute
- joint joint2: limit (none) -> lower=-3.14 upper=3.14 effort=30 velocity=1.0; type continuous -> revolute
