Commit message: Fix mit_humanoid_leg xacro

File: robot-models/mit_humanoid_leg.urdf (robot description, URDF)
Before this commit: robot mit_humanoid_leg, 11 links, 10 joints
Joints:
- joint base_to_hipz_link: limit (none) -> lower=-10 upper=10 effort=150 velocity=100; type continuous -> revolute
- joint base_to_hipz_rotor: limit (none) -> lower=-10 upper=10 effort=150 velocity=100; type continuous -> revolute
- joint hipx_to_hipy_link: limit (none) -> lower=-10 upper=10 effort=150 velocity=100; type continuous -> revolute
- joint hipx_to_hipy_rotor: limit (none) -> lower=-10 upper=10 effort=150 velocity=100; type continuous -> revolute
- joint hipy_to_ankle_rotor: limit (none) -> lower=-10 upper=10 effort=150 velocity=100; type continuous -> revolute
- joint hipy_to_knee_link: limit (none) -> lower=-10 upper=10 effort=150 velocity=100; type continuous -> revolute
- joint hipy_to_knee_rotor: limit (none) -> lower=-10 upper=10 effort=150 velocity=100; type continuous -> revolute
- joint hipz_to_hipx_link: limit (none) -> lower=-10 upper=10 effort=150 velocity=100; type continuous -> revolute
- joint hipz_to_hipx_rotor: limit (none) -> lower=-10 upper=10 effort=150 velocity=100; type continuous -> revolute
- joint knee_to_ankle: limit (none) -> lower=-10 upper=10 effort=150 velocity=100; type continuous -> revolute

File: robot-models/mit_humanoid_leg.xacro (robot description, xacro)
@@ -1,12 +1,18 @@
 <?xml version="1.0" ?>
 <robot name="mit_humanoid_leg" xmlns:xacro="http://ros.org/wiki/xacro">
+    <xacro:property name="effort_limit" value="150"/>
+    <xacro:property name="velocity_limit" value="100"/>
+    <xacro:property name="joint_lower_limit" value="-10"/>
+    <xacro:property name="joint_upper_limit" value="10"/>
     <!-- Hip Yaw Macro -->
     <xacro:property name="hipz_pitch" value="-0.174533"/>
     <xacro:macro name="hipz" params="prefix y_sign">
-        <joint name="base_to_${prefix}hipz_link" type="continuous">
+        <joint name="base_to_${prefix}hipz_link" type="revolute">
             <axis xyz="0 0 1"/>
             <origin xyz="-0.00565 ${y_sign * -0.082} -0.05735" rpy="0 ${hipz_pitch} 0"/>
             <parent link="base"/>
             <child link="${prefix}hip_rz_link"/>
+            <limit effort="${effort_limit}" velocity="${velocity_limit}"
+                   lower="${joint_lower_limit}" upper="${joint_upper_limit}"/>
         </joint>
         <link name="${prefix}hip_rz_link">
@@ -18,9 +24,11 @@
             </inertial>
         </link>
-        <joint name="${prefix}base_to_hipz_rotor" type="continuous" independent="false">
+        <joint name="${prefix}base_to_hipz_rotor" type="revolute" independent="false">
             <axis xyz="0 0 1"/>
             <origin xyz="-0.00842837 ${y_sign * -0.082} -0.041593" rpy="0 ${hipz_pitch} 0"/>
             <parent link="base"/>
             <child link="${prefix}hip_rz_rotor"/>
+            <limit effort="${effort_limit}" velocity="${velocity_limit}"
+                   lower="${joint_lower_limit}" upper="${joint_upper_limit}"/>
         </joint>
         <link name="${prefix}hip_rz_rotor">
@@ -41,9 +49,11 @@
     <xacro:property name="hipx_pitch" value="0.436332"/>
     <xacro:macro name="hipx" params="prefix y_sign">
-        <joint name="${prefix}hipz_to_hipx_link" type="continuous">
+        <joint name="${prefix}hipz_to_hipx_link" type="revolute">
             <axis xyz="1 0 0"/>
             <origin xyz="-0.06435 0.0 -.07499" rpy="0 ${hipx_pitch} 0"/>
             <parent link="${prefix}hip_rz_link"/>
             <child link="${prefix}hip_rx_link"/>
+            <limit effort="${effort_limit}" velocity="${velocity_limit}"
+                   lower="${joint_lower_limit}" upper="${joint_upper_limit}"/>
         </joint>
         <link name="${prefix}hip_rx_link">
@@ -55,9 +65,11 @@
             </inertial>
         </link>
-        <joint name="${prefix}hipz_to_hipx_rotor" type="continuous" independent="false">
+        <joint name="${prefix}hipz_to_hipx_rotor" type="revolute" independent="false">
             <axis xyz="1 0 0"/>
             <origin xyz="-0.0827 0.0 -0.066436" rpy="0 ${hipx_pitch} 0"/>
             <parent link="${prefix}hip_rz_link"/>
             <child link="${prefix}hip_rx_rotor"/>
+            <limit effort="${effort_limit}" velocity="${velocity_limit}"
+                   lower="${joint_lower_limit}" upper="${joint_upper_limit}"/>
         </joint>
         <link name="${prefix}hip_rx_rotor">
@@ -77,9 +89,11 @@
     <!-- Hip Flexion/Extension -->
     <xacro:macro name="hipy" params="prefix y_sign">
-        <joint name="${prefix}hipx_to_hipy_link" type="continuous">
+        <joint name="${prefix}hipx_to_hipy_link" type="revolute">
             <axis xyz="0 1 0"/>
             <origin xyz="0.071 ${y_sign * 0.0018375} 0.0" rpy="0 -${hipz_pitch + hipx_pitch} 0"/>
             <parent link="${prefix}hip_rx_link"/>
             <child link="${prefix}hip_ry_link"/>
+            <limit effort="${effort_limit}" velocity="${velocity_limit}"
+                   lower="${joint_lower_limit}" upper="${joint_upper_limit}"/>
         </joint>
         <link name="${prefix}hip_ry_link">
@@ -91,9 +105,11 @@
             </inertial>
         </link>
-        <joint name="${prefix}hipx_to_hipy_rotor" type="continuous" independent="false">
+        <joint name="${prefix}hipx_to_hipy_rotor" type="revolute" independent="false">
             <axis xyz="0 1 0"/>
             <origin xyz="0.071 ${y_sign * 0.024} 0.0" rpy="0 -${hipz_pitch + hipx_pitch} 0"/>
             <parent link="${prefix}hip_rx_link"/>
             <child link="${prefix}hip_ry_rotor"/>
+            <limit effort="${effort_limit}" velocity="${velocity_limit}"
+                   lower="${joint_lower_limit}" upper="${joint_upper_limit}"/>
         </joint>
         <link name="${prefix}hip_ry_rotor">
@@ -113,9 +129,11 @@
     <!-- Knee Flexion/Extension -->
     <xacro:macro name="knee" params="prefix y_sign">
-        <joint name="${prefix}hipy_to_knee_link" type="continuous">
+        <joint name="${prefix}hipy_to_knee_link" type="revolute">
             <axis xyz="0 1 0"/>
             <origin xyz="0.0 0.0 -0.267"/>
             <parent link="${prefix}hip_ry_link"/>
             <child link="${prefix}knee_link"/>
+            <limit effort="${effort_limit}" velocity="${velocity_limit}"
+                   lower="${joint_lower_limit}" upper="${joint_upper_limit}"/>
         </joint>
         <link name="${prefix}knee_link">
@@ -127,9 +145,11 @@
             </inertial>
         </link>
-        <joint name="${prefix}hipy_to_knee_rotor" type="continuous" independent="false">
+        <joint name="${prefix}hipy_to_knee_rotor" type="revolute" independent="false">
             <axis xyz="0 1 0"/>
             <origin xyz="0.013 ${y_sign * -0.0497} -0.0178"/>
             <parent link="${prefix}hip_ry_link"/>
             <child link="${prefix}knee_rotor"/>
+            <limit effort="${effort_limit}" velocity="${velocity_limit}"
+                   lower="${joint_lower_limit}" upper="${joint_upper_limit}"/>
         </joint>
         <link name="${prefix}knee_rotor">
@@ -149,23 +169,11 @@
     <!-- Ankle Flexion/Extension -->
     <xacro:macro name="ankle" params="prefix y_sign">
-        <joint name="${prefix}hipy_to_ankle_rotor" type="continuous" independent="false">
-            <axis xyz="0 1 0"/>
-            <origin xyz=".01563 ${y_sign * -.0454} -.13354"/>
-            <parent link="${prefix}hip_ry_link"/>
-            <child link="${prefix}ankle_rotor"/>
-        </joint>
-        <link name="${prefix}ankle_rotor">
-            <inertial>
-                <mass value="0."/>
-                <origin xyz="0. 0. 0."/>
-                <inertia ixx="1.084e-4" ixy="0.0" ixz="0.0"
-                         iyy="1.6841e-4" iyz="0.0" izz="1.084e-4"/>
-            </inertial>
-        </link>
-        <joint name="${prefix}knee_to_ankle" type="continuous">
+        <joint name="${prefix}knee_to_ankle" type="revolute">
             <axis xyz="0 1 0"/>
             <origin xyz="0.0 0.0 -0.2785"/>
             <parent link="${prefix}knee_link"/>
             <child link="${prefix}ankle_link"/>
+            <limit effort="${effort_limit}" velocity="${velocity_limit}"
+                   lower="${joint_lower_limit}" upper="${joint_upper_limit}"/>
         </joint>
         <link name="${prefix}ankle_link">
@@ -177,4 +185,20 @@
             </inertial>
         </link>
+        <joint name="${prefix}hipy_to_ankle_rotor" type="revolute" independent="false">
+            <axis xyz="0 1 0"/>
+            <origin xyz=".01563 ${y_sign * -.0454} -.13354"/>
+            <parent link="${prefix}hip_ry_link"/>
+            <child link="${prefix}ankle_rotor"/>
+            <limit effort="${effort_limit}" velocity="${velocity_limit}"
+                   lower="${joint_lower_limit}" upper="${joint_upper_limit}"/>
+        </joint>
+        <link name="${prefix}ankle_rotor">
+            <inertial>
+                <mass value="0."/>
+                <origin xyz="0. 0. 0."/>
+                <inertia ixx="1.084e-4" ixy="0.0" ixz="0.0"
+                         iyy="1.6841e-4" iyz="0.0" izz="1.084e-4"/>
+            </inertial>
+        </link>
         <constraint name="ankle_transmission" type="rolling">
             <predecessor link="${prefix}ankle_link"/>
@@ -184,8 +208,8 @@
     </xacro:macro>
     <link name="base"/>
-    <hipz prefix="" y_sign="1"/>
-    <hipx prefix="" y_sign="1"/>
-    <hipy prefix="" y_sign="1"/>
-    <knee prefix="" y_sign="1"/>
-    <ankle prefix="" y_sign="1"/>
+    <xacro:hipz prefix="" y_sign="1"/>
+    <xacro:hipx prefix="" y_sign="1"/>
+    <xacro:hipy prefix="" y_sign="1"/>
+    <xacro:knee prefix="" y_sign="1"/>
+    <xacro:ankle prefix="" y_sign="1"/>
 </robot>
