Commit message: Fix mini cheetah urdf

File: robot-models/mini_cheetah.urdf (robot description, URDF)
Before this commit: robot mini_cheetah, 25 links, 24 joints
Links:
- link FL_abad_rotor: mass 0. -> 0.055
- link FL_hip_rotor: mass 0. -> 0.055
- link FL_knee_rotor: mass 0. -> 0.055
- link FR_abad_rotor: mass 0. -> 0.055
- link FR_hip_rotor: mass 0. -> 0.055
- link FR_knee_rotor: mass 0. -> 0.055
- link HL_abad_rotor: mass 0. -> 0.055
- link HL_hip_rotor: mass 0. -> 0.055
- link HL_knee_rotor: mass 0. -> 0.055
- link HR_abad_rotor: mass 0. -> 0.055
- link HR_hip_rotor: mass 0. -> 0.055
- link HR_knee_rotor: mass 0. -> 0.055
Joints:
- joint FL_abad_to_hip_j: origin xyz=0 0.062 0.0 -> xyz=0 0.062 0.0 rpy=0 0 3.14159265359
- joint FL_abad_to_hip_rotor_j: origin xyz=0.0 0.04 0.0 rpy=0 0 0 -> xyz=0.0 0.04 0.0 rpy=0 0 3.14159265359
- joint FR_abad_to_hip_j: origin xyz=0 -0.062 0.0 -> xyz=0 -0.062 0.0 rpy=0 0 3.14159265359
- joint FR_abad_to_hip_rotor_j: origin xyz=0.0 -0.04 0.0 rpy=0 0 0 -> xyz=0.0 -0.04 0.0 rpy=0 0 3.14159265359
- joint HL_abad_to_hip_j: origin xyz=0 0.062 0.0 -> xyz=0 0.062 0.0 rpy=0 0 3.14159265359
- joint HL_abad_to_hip_rotor_j: origin xyz=0.0 0.04 0.0 rpy=0 0 0 -> xyz=0.0 0.04 0.0 rpy=0 0 3.14159265359
- joint HR_abad_to_hip_j: origin xyz=0 -0.062 0.0 -> xyz=0 -0.062 0.0 rpy=0 0 3.14159265359
- joint HR_abad_to_hip_rotor_j: origin xyz=0.0 -0.04 0.0 rpy=0 0 0 -> xyz=0.0 -0.04 0.0 rpy=0 0 3.14159265359
- joint torso_to_FL_abad_j: origin xyz=0.19 0.05 0.0 -> xyz=0.19 0.049 0.0
- joint torso_to_FR_abad_j: origin xyz=0.19 -0.05 0.0 -> xyz=0.19 -0.049 0.0
- joint torso_to_HL_abad_j: origin xyz=-0.19 0.05 0.0 -> xyz=-0.19 0.049 0.0
- joint torso_to_HR_abad_j: origin xyz=-0.19 -0.05 0.0 -> xyz=-0.19 -0.049 0.0

File: robot-models/mini_cheetah_fl_leg.urdf (robot description, URDF)
Before this commit: robot mini_cheetah_fl_leg, 7 links, 6 joints
Links:
- link FL_abad_rotor: mass 0. -> 0.055
- link FL_hip_rotor: mass 0. -> 0.055
- link FL_knee_rotor: mass 0. -> 0.055
Joints:
- joint FL_abad_to_hip_j: origin xyz=0 0.062 0.0 -> xyz=0 0.062 0.0 rpy=0 0 3.14159265359
- joint FL_abad_to_hip_rotor_j: origin xyz=0.0 0.04 0.0 rpy=0 0 0 -> xyz=0.0 0.04 0.0 rpy=0 0 3.14159265359
- joint torso_to_FL_abad_j: origin xyz=0.19 0.05 0.0 -> xyz=0.19 0.049 0.0

File: robot-models/mini_cheetah_fr_leg.urdf (robot description, URDF)
Before this commit: robot mini_cheetah_fr_leg, 7 links, 6 joints
Links:
- link FR_abad_rotor: mass 0. -> 0.055
- link FR_hip_rotor: mass 0. -> 0.055
- link FR_knee_rotor: mass 0. -> 0.055
Joints:
- joint FR_abad_to_hip_j: origin xyz=0 -0.062 0.0 -> xyz=0 -0.062 0.0 rpy=0 0 3.14159265359
- joint FR_abad_to_hip_rotor_j: origin xyz=0.0 -0.04 0.0 rpy=0 0 0 -> xyz=0.0 -0.04 0.0 rpy=0 0 3.14159265359
- joint torso_to_FR_abad_j: origin xyz=0.19 -0.05 0.0 -> xyz=0.19 -0.049 0.0

File: robot-models/mini_cheetah_hl_leg.urdf (robot description, URDF)
Before this commit: robot mini_cheetah_hl_leg, 7 links, 6 joints
Links:
- link HL_abad_rotor: mass 0. -> 0.055
- link HL_hip_rotor: mass 0. -> 0.055
- link HL_knee_rotor: mass 0. -> 0.055
Joints:
- joint HL_abad_to_hip_j: origin xyz=0 0.062 0.0 -> xyz=0 0.062 0.0 rpy=0 0 3.14159265359
- joint HL_abad_to_hip_rotor_j: origin xyz=0.0 0.04 0.0 rpy=0 0 0 -> xyz=0.0 0.04 0.0 rpy=0 0 3.14159265359
- joint torso_to_HL_abad_j: origin xyz=-0.19 0.05 0.0 -> xyz=-0.19 0.049 0.0

File: robot-models/mini_cheetah_hr_leg.urdf (robot description, URDF)
Before this commit: robot mini_cheetah_hr_leg, 7 links, 6 joints
Links:
- link HR_abad_rotor: mass 0. -> 0.055
- link HR_hip_rotor: mass 0. -> 0.055
- link HR_knee_rotor: mass 0. -> 0.055
Joints:
- joint HR_abad_to_hip_j: origin xyz=0 -0.062 0.0 -> xyz=0 -0.062 0.0 rpy=0 0 3.14159265359
- joint HR_abad_to_hip_rotor_j: origin xyz=0.0 -0.04 0.0 rpy=0 0 0 -> xyz=0.0 -0.04 0.0 rpy=0 0 3.14159265359
- joint torso_to_HR_abad_j: origin xyz=-0.19 -0.05 0.0 -> xyz=-0.19 -0.049 0.0

File: robot-models/mini_cheetah_properties.xacro (robot description, xacro)
@@ -1,9 +1,10 @@
 <?xml version="1.0" ?>
 <robot xmlns:xacro="http://ros.org/wiki/xacro">
+    <xacro:property name="u8_mass" value="0.055"/>
     <!-- Ab/Ad Macro -->
     <xacro:macro name="abad" params="prefix x_sign y_sign">
         <joint name="torso_to_${prefix}_abad_j" type="continuous">
             <axis xyz="1 0 0"/>
-            <origin xyz="${x_sign * 0.19} ${y_sign * 0.05} 0.0"/>
+            <origin xyz="${x_sign * 0.19} ${y_sign * 0.049} 0.0"/>
             <parent link="Floating Base"/>
             <child link="${prefix}_abad_link"/>
@@ -27,5 +28,5 @@
         <link name="${prefix}_abad_rotor">
             <inertial>
-                <mass value="0."/>
+                <mass value="${u8_mass}"/>
                 <origin xyz="0. 0. 0."/>
                 <inertia ixx="${63 * 1e-6}" ixy="0.0"
@@ -44,5 +45,5 @@
         <joint name="${prefix}_abad_to_hip_j" type="continuous">
             <axis xyz="0 1 0"/>
-            <origin xyz="0 ${y_sign * 0.062} 0.0"/>
+            <origin xyz="0 ${y_sign * 0.062} 0.0" rpy="0 0 ${pi}"/>
             <parent link="${prefix}_abad_link"/>
             <child link="${prefix}_hip_link"/>
@@ -60,5 +61,5 @@
         <joint name="${prefix}_abad_to_hip_rotor_j" type="continuous" independent="false">
             <axis xyz="0 1 0"/>
-            <origin rpy="0 0 0" xyz="0.0 ${y_sign * 0.04} 0.0"/>
+            <origin xyz="0.0 ${y_sign * 0.04} 0.0" rpy="0 0 ${pi}"/>
             <parent link="${prefix}_abad_link"/>
             <child link="${prefix}_hip_rotor"/>
@@ -66,5 +67,5 @@
         <link name="${prefix}_hip_rotor">
             <inertial>
-                <mass value="0."/>
+                <mass value="${u8_mass}"/>
                 <origin xyz="0. 0. 0."/>
                 <inertia ixx="${33 * 1e-6}" ixy="0.0"
@@ -91,7 +92,7 @@
                 <mass value="0.064"/>
                 <origin xyz="0.0 0.0 -0.061"/>
-                <inertia ixx="${6 * 1e-6}" ixy="0.0"
+                <inertia ixx="${245 * 1e-6}" ixy="0.0"
                          ixz="0.0" iyy="${248 * 1e-6}"
-                         iyz="0.0" izz="${245 * 1e-6}"/>
+                         iyz="0.0" izz="${6 * 1e-6}"/>
             </inertial>
             <!-- TODO(@MatthewChignoli): Do collision and visual stuff later -->
@@ -104,5 +105,5 @@
         <link name="${prefix}_knee_rotor">
             <inertial>
-                <mass value="0."/>
+                <mass value="${u8_mass}"/>
                 <origin xyz="0. 0. 0."/>
                 <inertia ixx="${33 * 1e-6}" ixy="0.0"

Commit message: Add double_pendulum, mini_cheetah, mit_humanoid into benchmark of explicit constrained systems

File: robot-models/mini_cheetah.urdf (robot description, URDF)
Before this commit: robot mini_cheetah, 25 links, 24 joints
Joints:
- joint FL_abad_to_hip_j: limit (none) -> lower=-10 upper=10 effort=150 velocity=100; origin xyz=0 0.062 0.0 rpy=0 0 3.14159265359 -> xyz=0 0.062 0.0 rpy=0 0 3.141592653589793; type continuous -> revolute
- joint FL_abad_to_hip_rotor_j: limit (none) -> lower=-10 upper=10 effort=150 velocity=100; origin xyz=0.0 0.04 0.0 rpy=0 0 3.14159265359 -> xyz=0.0 0.04 0.0 rpy=0 0 3.141592653589793; type continuous -> revolute
- joint FL_hip_to_knee_j: limit (none) -> lower=-10 upper=10 effort=150 velocity=100; type continuous -> revolute
- joint FL_hip_to_knee_rotor_j: limit (none) -> lower=-10 upper=10 effort=150 velocity=100; type continuous -> revolute
- joint FR_abad_to_hip_j: limit (none) -> lower=-10 upper=10 effort=150 velocity=100; origin xyz=0 -0.062 0.0 rpy=0 0 3.14159265359 -> xyz=0 -0.062 0.0 rpy=0 0 3.141592653589793; type continuous -> revolute
- joint FR_abad_to_hip_rotor_j: limit (none) -> lower=-10 upper=10 effort=150 velocity=100; origin xyz=0.0 -0.04 0.0 rpy=0 0 3.14159265359 -> xyz=0.0 -0.04 0.0 rpy=0 0 3.141592653589793; type continuous -> revolute
- joint FR_hip_to_knee_j: limit (none) -> lower=-10 upper=10 effort=150 velocity=100; type continuous -> revolute
- joint FR_hip_to_knee_rotor_j: limit (none) -> lower=-10 upper=10 effort=150 velocity=100; type continuous -> revolute
- joint HL_abad_to_hip_j: limit (none) -> lower=-10 upper=10 effort=150 velocity=100; origin xyz=0 0.062 0.0 rpy=0 0 3.14159265359 -> xyz=0 0.062 0.0 rpy=0 0 3.141592653589793; type continuous -> revolute
- joint HL_abad_to_hip_rotor_j: limit (none) -> lower=-10 upper=10 effort=150 velocity=100; origin xyz=0.0 0.04 0.0 rpy=0 0 3.14159265359 -> xyz=0.0 0.04 0.0 rpy=0 0 3.141592653589793; type continuous -> revolute
- joint HL_hip_to_knee_j: limit (none) -> lower=-10 upper=10 effort=150 velocity=100; type continuous -> revolute
- joint HL_hip_to_knee_rotor_j: limit (none) -> lower=-10 upper=10 effort=150 velocity=100; type continuous -> revolute
- joint HR_abad_to_hip_j: limit (none) -> lower=-10 upper=10 effort=150 velocity=100; origin xyz=0 -0.062 0.0 rpy=0 0 3.14159265359 -> xyz=0 -0.062 0.0 rpy=0 0 3.141592653589793; type continuous -> revolute
- joint HR_abad_to_hip_rotor_j: limit (none) -> lower=-10 upper=10 effort=150 velocity=100; origin xyz=0.0 -0.04 0.0 rpy=0 0 3.14159265359 -> xyz=0.0 -0.04 0.0 rpy=0 0 3.141592653589793; type continuous -> revolute
- joint HR_hip_to_knee_j: limit (none) -> lower=-10 upper=10 effort=150 velocity=100; type continuous -> revolute
- joint HR_hip_to_knee_rotor_j: limit (none) -> lower=-10 upper=10 effort=150 velocity=100; type continuous -> revolute
- joint torso_to_FL_abad_j: limit (none) -> lower=-10 upper=10 effort=150 velocity=100; type continuous -> revolute
- joint torso_to_FL_abad_rotor_j: limit (none) -> lower=-10 upper=10 effort=150 velocity=100; type continuous -> revolute
- joint torso_to_FR_abad_j: limit (none) -> lower=-10 upper=10 effort=150 velocity=100; type continuous -> revolute
- joint torso_to_FR_abad_rotor_j: limit (none) -> lower=-10 upper=10 effort=150 velocity=100; type continuous -> revolute
- joint torso_to_HL_abad_j: limit (none) -> lower=-10 upper=10 effort=150 velocity=100; type continuous -> revolute
- joint torso_to_HL_abad_rotor_j: limit (none) -> lower=-10 upper=10 effort=150 velocity=100; type continuous -> revolute
- joint torso_to_HR_abad_j: limit (none) -> lower=-10 upper=10 effort=150 velocity=100; type continuous -> revolute
- joint torso_to_HR_abad_rotor_j: limit (none) -> lower=-10 upper=10 effort=150 velocity=100; type continuous -> revolute

File: robot-models/mini_cheetah_properties.xacro (robot description, xacro)
@@ -2,11 +2,17 @@
 <robot xmlns:xacro="http://ros.org/wiki/xacro">
     <xacro:property name="u8_mass" value="0.055"/>
+    <xacro:property name="effort_limit" value="150"/>
+    <xacro:property name="velocity_limit" value="100"/>
+    <xacro:property name="joint_lower_limit" value="-10"/>
+    <xacro:property name="joint_upper_limit" value="10"/>
     <!-- Ab/Ad Macro -->
     <xacro:macro name="abad" params="prefix x_sign y_sign">
-        <joint name="torso_to_${prefix}_abad_j" type="continuous">
+        <joint name="torso_to_${prefix}_abad_j" type="revolute">
             <axis xyz="1 0 0"/>
             <origin xyz="${x_sign * 0.19} ${y_sign * 0.049} 0.0"/>
             <parent link="Floating Base"/>
             <child link="${prefix}_abad_link"/>
+            <limit effort="${effort_limit}" velocity="${velocity_limit}"
+                   lower="${joint_lower_limit}" upper="${joint_upper_limit}"/>
         </joint>
         <link name="${prefix}_abad_link">
@@ -20,9 +26,11 @@
             <!-- TODO(@MatthewChignoli): Do collision and visual stuff later -->
         </link>
-        <joint name="torso_to_${prefix}_abad_rotor_j" type="continuous" independent="false">
+        <joint name="torso_to_${prefix}_abad_rotor_j" type="revolute" independent="false">
             <axis xyz="1 0 0"/>
             <origin xyz="${x_sign * 0.125} ${y_sign * 0.049} 0.0"/>
             <parent link="Floating Base"/>
             <child link="${prefix}_abad_rotor"/>
+            <limit effort="${effort_limit}" velocity="${velocity_limit}"
+                   lower="${joint_lower_limit}" upper="${joint_upper_limit}"/>
         </joint>
         <link name="${prefix}_abad_rotor">
@@ -43,9 +51,11 @@
     <!-- Hip Macro -->
     <xacro:macro name="hip" params="prefix x_sign y_sign">
-        <joint name="${prefix}_abad_to_hip_j" type="continuous">
+        <joint name="${prefix}_abad_to_hip_j" type="revolute">
             <axis xyz="0 1 0"/>
             <origin xyz="0 ${y_sign * 0.062} 0.0" rpy="0 0 ${pi}"/>
             <parent link="${prefix}_abad_link"/>
             <child link="${prefix}_hip_link"/>
+            <limit effort="${effort_limit}" velocity="${velocity_limit}"
+                   lower="${joint_lower_limit}" upper="${joint_upper_limit}"/>
         </joint>
         <link name="${prefix}_hip_link">
@@ -59,9 +69,11 @@
             <!-- TODO(@MatthewChignoli): Do collision and visual stuff later -->
         </link>
-        <joint name="${prefix}_abad_to_hip_rotor_j" type="continuous" independent="false">
+        <joint name="${prefix}_abad_to_hip_rotor_j" type="revolute" independent="false">
             <axis xyz="0 1 0"/>
             <origin xyz="0.0 ${y_sign * 0.04} 0.0" rpy="0 0 ${pi}"/>
             <parent link="${prefix}_abad_link"/>
             <child link="${prefix}_hip_rotor"/>
+            <limit effort="${effort_limit}" velocity="${velocity_limit}"
+                   lower="${joint_lower_limit}" upper="${joint_upper_limit}"/>
         </joint>
         <link name="${prefix}_hip_rotor">
@@ -82,9 +94,11 @@
     <!-- Knee Macro -->
     <xacro:macro name="knee" params="prefix x_sign y_sign">
-        <joint name="${prefix}_hip_to_knee_j" type="continuous">
+        <joint name="${prefix}_hip_to_knee_j" type="revolute">
             <axis xyz="0 1 0"/>
             <origin xyz="0.0 0.0 -0.209"/>
             <parent link="${prefix}_hip_link"/>
             <child link="${prefix}_knee_link"/>
+            <limit effort="${effort_limit}" velocity="${velocity_limit}"
+                   lower="${joint_lower_limit}" upper="${joint_upper_limit}"/>
         </joint>
         <link name="${prefix}_knee_link">
@@ -98,8 +112,10 @@
             <!-- TODO(@MatthewChignoli): Do collision and visual stuff later -->
         </link>
-        <joint name="${prefix}_hip_to_knee_rotor_j" type="continuous" independent="false">
+        <joint name="${prefix}_hip_to_knee_rotor_j" type="revolute" independent="false">
             <axis xyz="0 1 0"/>
             <parent link="${prefix}_hip_link"/>
             <child link="${prefix}_knee_rotor"/>
+            <limit effort="${effort_limit}" velocity="${velocity_limit}"
+                   lower="${joint_lower_limit}" upper="${joint_upper_limit}"/>
         </joint>
         <link name="${prefix}_knee_rotor">

File: robot-models/mit_humanoid.urdf (robot description, URDF)
Before this commit: robot mit_humanoid, 37 links, 36 joints
Joints:
- joint base_to_left_hipz_link: limit (none) -> lower=-10 upper=10 effort=150 velocity=100; type continuous -> revolute
- joint base_to_left_shouldery_link: limit (none) -> lower=-10 upper=10 effort=150 velocity=100; type continuous -> revolute
- joint base_to_left_shouldery_rotor: limit (none) -> lower=-10 upper=10 effort=150 velocity=100; type continuous -> revolute
- joint base_to_right_hipz_link: limit (none) -> lower=-10 upper=10 effort=150 velocity=100; type continuous -> revolute
- joint base_to_right_shouldery_link: limit (none) -> lower=-10 upper=10 effort=150 velocity=100; type continuous -> revolute
- joint base_to_right_shouldery_rotor: limit (none) -> lower=-10 upper=10 effort=150 velocity=100; type continuous -> revolute
- joint left_base_to_hipz_rotor: limit (none) -> lower=-10 upper=10 effort=150 velocity=100; type continuous -> revolute
- joint left_hipx_to_hipy_link: limit (none) -> lower=-10 upper=10 effort=150 velocity=100; type continuous -> revolute
- joint left_hipx_to_hipy_rotor: limit (none) -> lower=-10 upper=10 effort=150 velocity=100; type continuous -> revolute
- joint left_hipy_to_ankle_rotor: limit (none) -> lower=-10 upper=10 effort=150 velocity=100; type continuous -> revolute
- joint left_hipy_to_knee_link: limit (none) -> lower=-10 upper=10 effort=150 velocity=100; type continuous -> revolute
- joint left_hipy_to_knee_rotor: limit (none) -> lower=-10 upper=10 effort=150 velocity=100; type continuous -> revolute
- joint left_hipz_to_hipx_link: limit (none) -> lower=-10 upper=10 effort=150 velocity=100; type continuous -> revolute
- joint left_hipz_to_hipx_rotor: limit (none) -> lower=-10 upper=10 effort=150 velocity=100; type continuous -> revolute
- joint left_knee_to_ankle: limit (none) -> lower=-10 upper=10 effort=150 velocity=100; type continuous -> revolute
- joint left_shoulderx_shoulderz_link: limit (none) -> lower=-10 upper=10 effort=150 velocity=100; type continuous -> revolute
- joint left_shoulderx_to_shoulderz_rotor: limit (none) -> lower=-10 upper=10 effort=150 velocity=100; type continuous -> revolute
- joint left_shouldery_shoulderx_link: limit (none) -> lower=-10 upper=10 effort=150 velocity=100; type continuous -> revolute
- joint left_shouldery_to_shoulderx_rotor: limit (none) -> lower=-10 upper=10 effort=150 velocity=100; type continuous -> revolute
- joint left_shoulderz_elbow_link: limit (none) -> lower=-10 upper=10 effort=150 velocity=100; type continuous -> revolute
- joint left_shoulderz_to_elbow_rotor: limit (none) -> lower=-10 upper=10 effort=150 velocity=100; type continuous -> revolute
- joint right_base_to_hipz_rotor: limit (none) -> lower=-10 upper=10 effort=150 velocity=100; type continuous -> revolute
- joint right_hipx_to_hipy_link: limit (none) -> lower=-10 upper=10 effort=150 velocity=100; type continuous -> revolute
- joint right_hipx_to_hipy_rotor: limit (none) -> lower=-10 upper=10 effort=150 velocity=100; type continuous -> revolute
- joint right_hipy_to_ankle_rotor: limit (none) -> lower=-10 upper=10 effort=150 velocity=100; type continuous -> revolute
- joint right_hipy_to_knee_link: limit (none) -> lower=-10 upper=10 effort=150 velocity=100; type continuous -> revolute
- joint right_hipy_to_knee_rotor: limit (none) -> lower=-10 upper=10 effort=150 velocity=100; type continuous -> revolute
- joint right_hipz_to_hipx_link: limit (none) -> lower=-10 upper=10 effort=150 velocity=100; type continuous -> revolute
- joint right_hipz_to_hipx_rotor: limit (none) -> lower=-10 upper=10 effort=150 velocity=100; type continuous -> revolute
- joint right_knee_to_ankle: limit (none) -> lower=-10 upper=10 effort=150 velocity=100; type continuous -> revolute
- joint right_shoulderx_shoulderz_link: limit (none) -> lower=-10 upper=10 effort=150 velocity=100; type continuous -> revolute
- joint right_shoulderx_to_shoulderz_rotor: limit (none) -> lower=-10 upper=10 effort=150 velocity=100; type continuous -> revolute
- joint right_shouldery_shoulderx_link: limit (none) -> lower=-10 upper=10 effort=150 velocity=100; type continuous -> revolute
- joint right_shouldery_to_shoulderx_rotor: limit (none) -> lower=-10 upper=10 effort=150 velocity=100; type continuous -> revolute
- joint right_shoulderz_elbow_link: limit (none) -> lower=-10 upper=10 effort=150 velocity=100; type continuous -> revolute
- joint right_shoulderz_to_elbow_rotor: limit (none) -> lower=-10 upper=10 effort=150 velocity=100; type continuous -> revolute
