Commit message: Add double_pendulum, mini_cheetah, mit_humanoid into benchmark of explicit constrained systems

File: robot-models/mit_humanoid.xacro (robot description, xacro)
@@ -1,12 +1,18 @@
 <?xml version="1.0" ?>
 <robot name="mit_humanoid" xmlns:xacro="http://ros.org/wiki/xacro">
+    <xacro:property name="effort_limit" value="150"/>
+    <xacro:property name="velocity_limit" value="100"/>
+    <xacro:property name="joint_lower_limit" value="-10"/>
+    <xacro:property name="joint_upper_limit" value="10"/>
     <!-- Hip Yaw Macro -->
     <xacro:property name="hipz_pitch" value="-0.174533"/>
     <xacro:macro name="hipz" params="prefix y_sign">
-        <joint name="base_to_${prefix}hipz_link" type="continuous">
+        <joint name="base_to_${prefix}hipz_link" type="revolute">
             <axis xyz="0 0 1"/>
             <origin xyz="-0.00565 ${y_sign * -0.082} -0.05735" rpy="0 ${hipz_pitch} 0"/>
             <parent link="Floating Base"/>
             <child link="${prefix}hip_rz_link"/>
+            <limit effort="${effort_limit}" velocity="${velocity_limit}"
+                   lower="${joint_lower_limit}" upper="${joint_upper_limit}"/>
         </joint>
         <link name="${prefix}hip_rz_link">
@@ -18,9 +24,11 @@
             </inertial>
         </link>
-        <joint name="${prefix}base_to_hipz_rotor" type="continuous" independent="false">
+        <joint name="${prefix}base_to_hipz_rotor" type="revolute" independent="false">
             <axis xyz="0 0 1"/>
             <origin xyz="-0.00842837 ${y_sign * -0.082} -0.041593" rpy="0 ${hipz_pitch} 0"/>
             <parent link="Floating Base"/>
             <child link="${prefix}hip_rz_rotor"/>
+            <limit effort="${effort_limit}" velocity="${velocity_limit}"
+                   lower="${joint_lower_limit}" upper="${joint_upper_limit}"/>
         </joint>
         <link name="${prefix}hip_rz_rotor">
@@ -41,9 +49,11 @@
     <xacro:property name="hipx_pitch" value="0.436332"/>
     <xacro:macro name="hipx" params="prefix y_sign">
-        <joint name="${prefix}hipz_to_hipx_link" type="continuous">
+        <joint name="${prefix}hipz_to_hipx_link" type="revolute">
             <axis xyz="1 0 0"/>
             <origin xyz="-0.06435 0.0 -.07499" rpy="0 ${hipx_pitch} 0"/>
             <parent link="${prefix}hip_rz_link"/>
             <child link="${prefix}hip_rx_link"/>
+            <limit effort="${effort_limit}" velocity="${velocity_limit}"
+                   lower="${joint_lower_limit}" upper="${joint_upper_limit}"/>
         </joint>
         <link name="${prefix}hip_rx_link">
@@ -55,9 +65,11 @@
             </inertial>
         </link>
-        <joint name="${prefix}hipz_to_hipx_rotor" type="continuous" independent="false">
+        <joint name="${prefix}hipz_to_hipx_rotor" type="revolute" independent="false">
             <axis xyz="1 0 0"/>
             <origin xyz="-0.0827 0.0 -0.066436" rpy="0 ${hipx_pitch} 0"/>
             <parent link="${prefix}hip_rz_link"/>
             <child link="${prefix}hip_rx_rotor"/>
+            <limit effort="${effort_limit}" velocity="${velocity_limit}"
+                   lower="${joint_lower_limit}" upper="${joint_upper_limit}"/>
         </joint>
         <link name="${prefix}hip_rx_rotor">
@@ -77,9 +89,11 @@
     <!-- Hip Flexion/Extension -->
     <xacro:macro name="hipy" params="prefix y_sign">
-        <joint name="${prefix}hipx_to_hipy_link" type="continuous">
+        <joint name="${prefix}hipx_to_hipy_link" type="revolute">
             <axis xyz="0 1 0"/>
             <origin xyz="0.071 ${y_sign * 0.0018375} 0.0" rpy="0 -${hipz_pitch + hipx_pitch} 0"/>
             <parent link="${prefix}hip_rx_link"/>
             <child link="${prefix}hip_ry_link"/>
+            <limit effort="${effort_limit}" velocity="${velocity_limit}"
+                   lower="${joint_lower_limit}" upper="${joint_upper_limit}"/>
         </joint>
         <link name="${prefix}hip_ry_link">
@@ -91,9 +105,11 @@
             </inertial>
         </link>
-        <joint name="${prefix}hipx_to_hipy_rotor" type="continuous" independent="false">
+        <joint name="${prefix}hipx_to_hipy_rotor" type="revolute" independent="false">
             <axis xyz="0 1 0"/>
             <origin xyz="0.071 ${y_sign * 0.024} 0.0" rpy="0 -${hipz_pitch + hipx_pitch} 0"/>
             <parent link="${prefix}hip_rx_link"/>
             <child link="${prefix}hip_ry_rotor"/>
+            <limit effort="${effort_limit}" velocity="${velocity_limit}"
+                   lower="${joint_lower_limit}" upper="${joint_upper_limit}"/>
         </joint>
         <link name="${prefix}hip_ry_rotor">
@@ -113,9 +129,11 @@
     <!-- Knee Flexion/Extension -->
     <xacro:macro name="knee" params="prefix y_sign">
-        <joint name="${prefix}hipy_to_knee_link" type="continuous">
+        <joint name="${prefix}hipy_to_knee_link" type="revolute">
             <axis xyz="0 1 0"/>
             <origin xyz="0.0 0.0 -0.267"/>
             <parent link="${prefix}hip_ry_link"/>
             <child link="${prefix}knee_link"/>
+            <limit effort="${effort_limit}" velocity="${velocity_limit}"
+                   lower="${joint_lower_limit}" upper="${joint_upper_limit}"/>
         </joint>
         <link name="${prefix}knee_link">
@@ -127,9 +145,11 @@
             </inertial>
         </link>
-        <joint name="${prefix}hipy_to_knee_rotor" type="continuous" independent="false">
+        <joint name="${prefix}hipy_to_knee_rotor" type="revolute" independent="false">
             <axis xyz="0 1 0"/>
             <origin xyz="0.013 ${y_sign * -0.0497} -0.0178"/>
             <parent link="${prefix}hip_ry_link"/>
             <child link="${prefix}knee_rotor"/>
+            <limit effort="${effort_limit}" velocity="${velocity_limit}"
+                   lower="${joint_lower_limit}" upper="${joint_upper_limit}"/>
         </joint>
         <link name="${prefix}knee_rotor">
@@ -149,9 +169,11 @@
     <!-- Ankle Flexion/Extension -->
     <xacro:macro name="ankle" params="prefix y_sign">
-        <joint name="${prefix}hipy_to_ankle_rotor" type="continuous" independent="false">
+        <joint name="${prefix}hipy_to_ankle_rotor" type="revolute" independent="false">
             <axis xyz="0 1 0"/>
             <origin xyz=".01563 ${y_sign * -.0454} -.13354"/>
             <parent link="${prefix}hip_ry_link"/>
             <child link="${prefix}ankle_rotor"/>
+            <limit effort="${effort_limit}" velocity="${velocity_limit}"
+                   lower="${joint_lower_limit}" upper="${joint_upper_limit}"/>
         </joint>
         <link name="${prefix}ankle_rotor">
@@ -163,9 +185,11 @@
             </inertial>
         </link>
-        <joint name="${prefix}knee_to_ankle" type="continuous">
+        <joint name="${prefix}knee_to_ankle" type="revolute">
             <axis xyz="0 1 0"/>
             <origin xyz="0.0 0.0 -0.2785"/>
             <parent link="${prefix}knee_link"/>
             <child link="${prefix}ankle_link"/>
+            <limit effort="${effort_limit}" velocity="${velocity_limit}"
+                   lower="${joint_lower_limit}" upper="${joint_upper_limit}"/>
         </joint>
         <link name="${prefix}ankle_link">
@@ -185,9 +209,11 @@
     <!-- Shoulder Y-axis -->
     <xacro:macro name="shouldery" params="prefix y_sign">
-        <joint name="base_to_${prefix}shouldery_link" type="continuous">
+        <joint name="base_to_${prefix}shouldery_link" type="revolute">
             <axis xyz="0 1 0"/>
             <origin xyz="0.01346 ${y_sign * -0.17608} 0.24657"/>
             <parent link="Floating Base"/>
             <child link="${prefix}shoulder_ry_link"/>
+            <limit effort="${effort_limit}" velocity="${velocity_limit}"
+                   lower="${joint_lower_limit}" upper="${joint_upper_limit}"/>
         </joint>
         <link name="${prefix}shoulder_ry_link">
@@ -199,9 +225,11 @@
             </inertial>
         </link>
-        <joint name="base_to_${prefix}shouldery_rotor" type="continuous" independent="false">
+        <joint name="base_to_${prefix}shouldery_rotor" type="revolute" independent="false">
             <axis xyz="0 1 0"/>
             <origin xyz="0.01346 ${y_sign * -0.16} 0.24657"/>
             <parent link="Floating Base"/>
             <child link="${prefix}shoulder_ry_rotor"/>
+            <limit effort="${effort_limit}" velocity="${velocity_limit}"
+                   lower="${joint_lower_limit}" upper="${joint_upper_limit}"/>
         </joint>
         <link name="${prefix}shoulder_ry_rotor">
@@ -221,9 +249,11 @@
     <!-- Shoulder X-axis -->
     <xacro:macro name="shoulderx" params="prefix y_sign">
-        <joint name="${prefix}shouldery_shoulderx_link" type="continuous">
+        <joint name="${prefix}shouldery_shoulderx_link" type="revolute">
             <axis xyz="1 0 0"/>
             <origin xyz="0. ${y_sign * -0.0575} 0."/>
             <parent link="${prefix}shoulder_ry_link"/>
             <child link="${prefix}shoulder_rx_link"/>
+            <limit effort="${effort_limit}" velocity="${velocity_limit}"
+                   lower="${joint_lower_limit}" upper="${joint_upper_limit}"/>
         </joint>
         <link name="${prefix}shoulder_rx_link">
@@ -235,9 +265,11 @@
             </inertial>
         </link>
-        <joint name="${prefix}shouldery_to_shoulderx_rotor" type="continuous" independent="false">
+        <joint name="${prefix}shouldery_to_shoulderx_rotor" type="revolute" independent="false">
             <axis xyz="1 0 0"/>
             <origin xyz="0. ${y_sign * -0.0575} 0."/>
             <parent link="${prefix}shoulder_ry_link"/>
             <child link="${prefix}shoulder_rx_rotor"/>
+            <limit effort="${effort_limit}" velocity="${velocity_limit}"
+                   lower="${joint_lower_limit}" upper="${joint_upper_limit}"/>
         </joint>
         <link name="${prefix}shoulder_rx_rotor">
@@ -257,9 +289,11 @@
     <!-- Shoulder Z-axis -->
     <xacro:macro name="shoulderz" params="prefix y_sign">
-        <joint name="${prefix}shoulderx_shoulderz_link" type="continuous">
+        <joint name="${prefix}shoulderx_shoulderz_link" type="revolute">
             <axis xyz="0 0 1"/>
             <origin xyz="0. ${y_sign * 0.} -0.10250"/>
             <parent link="${prefix}shoulder_rx_link"/>
             <child link="${prefix}shoulder_rz_link"/>
+            <limit effort="${effort_limit}" velocity="${velocity_limit}"
+                   lower="${joint_lower_limit}" upper="${joint_upper_limit}"/>
         </joint>
         <link name="${prefix}shoulder_rz_link">
@@ -271,9 +305,11 @@
             </inertial>
         </link>
-        <joint name="${prefix}shoulderx_to_shoulderz_rotor" type="continuous" independent="false">
+        <joint name="${prefix}shoulderx_to_shoulderz_rotor" type="revolute" independent="false">
             <axis xyz="0 0 1"/>
             <origin xyz="0. ${y_sign * 0.} -0.10250"/>
             <parent link="${prefix}shoulder_rx_link"/>
             <child link="${prefix}shoulder_rz_rotor"/>
+            <limit effort="${effort_limit}" velocity="${velocity_limit}"
+                   lower="${joint_lower_limit}" upper="${joint_upper_limit}"/>
         </joint>
         <link name="${prefix}shoulder_rz_rotor">
@@ -293,9 +329,11 @@
     <!-- Elbow Flexion/Extension -->
     <xacro:macro name="elbow" params="prefix y_sign">
-        <joint name="${prefix}shoulderz_elbow_link" type="continuous">
+        <joint name="${prefix}shoulderz_elbow_link" type="revolute">
             <axis xyz="0 1 0"/>
             <origin xyz="0. ${y_sign * 0.} -0.1455"/>
             <parent link="${prefix}shoulder_rz_link"/>
             <child link="${prefix}elbow_link"/>
+            <limit effort="${effort_limit}" velocity="${velocity_limit}"
+                   lower="${joint_lower_limit}" upper="${joint_upper_limit}"/>
         </joint>
         <link name="${prefix}elbow_link">
@@ -307,9 +345,11 @@
             </inertial>
         </link>
-        <joint name="${prefix}shoulderz_to_elbow_rotor" type="continuous" independent="false">
+        <joint name="${prefix}shoulderz_to_elbow_rotor" type="revolute" independent="false">
             <axis xyz="0 1 0"/>
             <origin xyz="0. ${y_sign * 0.0325} -0.06"/>
             <parent link="${prefix}shoulder_rz_link"/>
             <child link="${prefix}elbow_rotor"/>
+            <limit effort="${effort_limit}" velocity="${velocity_limit}"
+                   lower="${joint_lower_limit}" upper="${joint_upper_limit}"/>
         </joint>
         <link name="${prefix}elbow_rotor">
@@ -336,21 +376,21 @@
         </inertial>
     </link>
-    <hipz prefix="right_" y_sign="1"/>
-    <hipz prefix="left_" y_sign="-1"/>
-    <hipx prefix="right_" y_sign="1"/>
-    <hipx prefix="left_" y_sign="-1"/>
-    <hipy prefix="right_" y_sign="1"/>
-    <hipy prefix="left_" y_sign="-1"/>
-    <knee prefix="right_" y_sign="1"/>
-    <knee prefix="left_" y_sign="-1"/>
-    <ankle prefix="right_" y_sign="1"/>
-    <ankle prefix="left_" y_sign="-1"/>
-    <shouldery prefix="right_" y_sign="1"/>
-    <shouldery prefix="left_" y_sign="-1"/>
-    <shoulderx prefix="right_" y_sign="1"/>
-    <shoulderx prefix="left_" y_sign="-1"/>
-    <shoulderz prefix="right_" y_sign="1"/>
-    <shoulderz prefix="left_" y_sign="-1"/>
-    <elbow prefix="right_" y_sign="1"/>
-    <elbow prefix="left_" y_sign="-1"/>
+    <xacro:hipz prefix="right_" y_sign="1"/>
+    <xacro:hipz prefix="left_" y_sign="-1"/>
+    <xacro:hipx prefix="right_" y_sign="1"/>
+    <xacro:hipx prefix="left_" y_sign="-1"/>
+    <xacro:hipy prefix="right_" y_sign="1"/>
+    <xacro:hipy prefix="left_" y_sign="-1"/>
+    <xacro:knee prefix="right_" y_sign="1"/>
+    <xacro:knee prefix="left_" y_sign="-1"/>
+    <xacro:ankle prefix="right_" y_sign="1"/>
+    <xacro:ankle prefix="left_" y_sign="-1"/>
+    <xacro:shouldery prefix="right_" y_sign="1"/>
+    <xacro:shouldery prefix="left_" y_sign="-1"/>
+    <xacro:shoulderx prefix="right_" y_sign="1"/>
+    <xacro:shoulderx prefix="left_" y_sign="-1"/>
+    <xacro:shoulderz prefix="right_" y_sign="1"/>
+    <xacro:shoulderz prefix="left_" y_sign="-1"/>
+    <xacro:elbow prefix="right_" y_sign="1"/>
+    <xacro:elbow prefix="left_" y_sign="-1"/>
 </robot>
