Commit message: WIP testing forward dynamics on Generic joints model vs pinocchio

File: robot-models/four_bar.urdf (robot description, URDF)
Before this commit: robot four_bar, 4 links, 3 joints
Joints:
- joint joint1: limit (none) -> lower=-3.14 upper=3.14 effort=30 velocity=1.0; type continuous -> revolute
- joint joint2: limit (none) -> lower=-3.14 upper=3.14 effort=30 velocity=1.0; origin xyz=0.1 0.0 0.0 -> xyz=0.2 0.0 0.0; type continuous -> revolute
- joint joint3: limit (none) -> lower=-3.14 upper=3.14 effort=30 velocity=1.0; type continuous -> revolute

File: robot-models/revolute_rotor_chain.urdf (robot description, URDF)
Before this commit: robot revolute_rotor_chain, 7 links, 6 joints
Joints:
- joint joint1: limit (none) -> lower=-10 upper=10 effort=30 velocity=1.0; type continuous -> revolute
- joint joint1r: limit (none) -> lower=-10 upper=10 effort=30 velocity=1.0; type continuous -> revolute
- joint joint2: limit (none) -> lower=-10 upper=10 effort=30 velocity=1.0; type continuous -> revolute
- joint joint2r: limit (none) -> lower=-10 upper=10 effort=30 velocity=1.0; type continuous -> revolute
- joint joint3: limit (none) -> lower=-10 upper=10 effort=30 velocity=1.0; type continuous -> revolute
- joint joint3r: limit (none) -> lower=-10 upper=10 effort=30 velocity=1.0; type continuous -> revolute

Commit message: Explicit benchmark works as expected

File: robot-models/four_bar.urdf (robot description, URDF)
Before this commit: robot four_bar, 4 links, 3 joints
Links:
- link link1: geometry visual box size=0.5 0.05 0.05
- link link2: geometry visual box size=1.0 0.05 0.05
- link link3: geometry visual box size=0.5 0.05 0.05
Joints:
- joint joint2: origin xyz=0.2 0.0 0.0 -> xyz=0.5 0.0 0.0
- joint joint3: origin xyz=0.0 0.0 0.0 -> xyz=1.0 0.0 0.0

Commit message: Pretty hacky, but implicit unit test passing

File: robot-models/four_bar.urdf (robot description, URDF)
Before this commit: robot four_bar, 4 links, 3 joints
Joints:
- joint joint1: limit lower=-3.14 upper=3.14 effort=30 velocity=1.0 -> lower=-13.14 upper=13.14 effort=30 velocity=1.0
- joint joint2: limit lower=-3.14 upper=3.14 effort=30 velocity=1.0 -> lower=-13.14 upper=13.14 effort=30 velocity=1.0
- joint joint3: limit lower=-3.14 upper=3.14 effort=30 velocity=1.0 -> lower=-13.14 upper=13.14 effort=30 velocity=1.0
