Commit message: Fix joint macro independent param

File: robot-models/revolute_rotor_chain.xacro (robot description, xacro)
@@ -9,6 +9,20 @@
     <xacro:property name="link_mass" value="1"/>
     <xacro:property name="rotor_mass" value="0"/>
-    <xacro:macro name="joint" params="name parent child independent=true">
-        <joint name="${name}" type="revolute" independent="${independent}">
+    <!-- NOTE(@nicholasadr): Had to separate independent and dependent joint macro
+                             because urdf will capitalize the first letter of boolean
+                             parameter "true/false" to "True/False", leading to
+                             incorrect joint registration -->
+    <xacro:macro name="independent_joint" params="name parent child">
+        <joint name="${name}" type="revolute" independent="true">
+            <parent link="${parent}"/>
+            <child link="${child}"/>
+            <axis xyz="0 0 1"/>
+            <origin xyz="1.0 0.0 0.0"/>
+            <limit effort="${effort_limit}" velocity="${velocity_limit}"
+                   lower="${joint_lower_limit}" upper="${joint_upper_limit}"/>
+        </joint>
+    </xacro:macro>
+    <xacro:macro name="dependent_joint" params="name parent child">
+        <joint name="${name}" type="revolute" independent="false">
             <parent link="${parent}"/>
             <child link="${child}"/>
@@ -45,7 +59,7 @@
     </xacro:macro>
     <xacro:macro name="base_chain">
-        <xacro:joint name="base_to_link_1" parent="base" child="link_1"/>
+        <xacro:independent_joint name="base_to_link_1" parent="base" child="link_1"/>
         <xacro:link name="link_1"/>
-        <xacro:joint name="base_to_rotor_1" parent="base" child="rotor_1" independent="false"/>
+        <xacro:dependent_joint name="base_to_rotor_1" parent="base" child="rotor_1"/>
         <xacro:rotor name="rotor_1"/>
         <xacro:transmission name="transmission_1" predecessor="link_1" successor="rotor_1"/>
@@ -53,7 +67,7 @@
     <xacro:macro name="revolute_rotor_loop" params="idx">
         <xacro:if value="${idx - 1}">
-            <xacro:joint name="link_${idx - 1}_to_link_${idx}" parent="link_${idx - 1}" child="link_${idx}"/>
+            <xacro:independent_joint name="link_${idx - 1}_to_link_${idx}" parent="link_${idx - 1}" child="link_${idx}"/>
             <xacro:link name="link_${idx}"/>
-            <xacro:joint name="link_${idx - 1}_to_rotor_${idx}" parent="base" child="rotor_${idx}" independent="false"/>
+            <xacro:dependent_joint name="link_${idx - 1}_to_rotor_${idx}" parent="base" child="rotor_${idx}"/>
             <xacro:rotor name="rotor_${idx}"/>
             <xacro:transmission name="transmission_${idx}" predecessor="link_${idx}" successor="rotor_${idx}"/>

File: robot-models/revolute_rotor_parallel.xacro (robot description, xacro)
@@ -9,6 +9,20 @@
     <xacro:property name="link_mass" value="0.1"/>
     <xacro:property name="rotor_mass" value="0.05"/>
-    <xacro:macro name="joint" params="name parent child independent=true">
-        <joint name="${name}" type="revolute" independent="${independent}">
+    <!-- NOTE(@nicholasadr): Had to separate independent and dependent joint macro
+                             because urdf will capitalize the first letter of boolean
+                             parameter "true/false" to "True/False", leading to
+                             incorrect joint registration -->
+    <xacro:macro name="independent_joint" params="name parent child">
+        <joint name="${name}" type="revolute" independent="true">
+            <parent link="${parent}"/>
+            <child link="${child}"/>
+            <axis xyz="0 0 1"/>
+            <origin xyz="1.0 0.0 0.0"/>
+            <limit effort="${effort_limit}" velocity="${velocity_limit}"
+                   lower="${joint_lower_limit}" upper="${joint_upper_limit}"/>
+        </joint>
+    </xacro:macro>
+    <xacro:macro name="dependent_joint" params="name parent child">
+        <joint name="${name}" type="revolute" independent="false">
             <parent link="${parent}"/>
             <child link="${child}"/>
@@ -45,7 +59,7 @@
     </xacro:macro>
     <xacro:macro name="base_chain">
-        <xacro:joint name="base_to_link_1" parent="base" child="link_1"/>
+        <xacro:independent_joint name="base_to_link_1" parent="base" child="link_1"/>
         <xacro:link name="link_1"/>
-        <xacro:joint name="base_to_rotor_1" parent="base" child="rotor_1" independent="false"/>
+        <xacro:dependent_joint name="base_to_rotor_1" parent="base" child="rotor_1"/>
         <xacro:rotor name="rotor_1"/>
         <xacro:transmission name="transmission_1" predecessor="link_1" successor="rotor_1"/>
@@ -53,7 +67,7 @@
     <xacro:macro name="revolute_rotor_loop" params="idx">
         <xacro:if value="${idx - 1}">
-            <xacro:joint name="link_${idx - 1}_to_link_${idx}" parent="link_${idx - 1}" child="link_${idx}"/>
+            <xacro:independent_joint name="link_${idx - 1}_to_link_${idx}" parent="link_${idx - 1}" child="link_${idx}"/>
             <xacro:link name="link_${idx}"/>
-            <xacro:joint name="base_to_rotor_${idx}" parent="base" child="rotor_${idx}" independent="false"/>
+            <xacro:dependent_joint name="base_to_rotor_${idx}" parent="base" child="rotor_${idx}"/>
             <xacro:rotor name="rotor_${idx}"/>
             <xacro:transmission name="transmission_${idx}" predecessor="link_${idx}" successor="rotor_${idx}"/>

Commit message: Systemize revolute rotor xacro

File: robot-models/revolute_rotor_chain.xacro (robot description, xacro)
@@ -3,78 +3,7 @@
     <xacro:arg name="loop_count" default="3"/>
     <xacro:property name="loop_count" value="$(arg loop_count)"/>
-    <xacro:property name="effort_limit" value="30"/>
-    <xacro:property name="velocity_limit" value="1.0"/>
-    <xacro:property name="joint_lower_limit" value="-10"/>
-    <xacro:property name="joint_upper_limit" value="10"/>
-    <xacro:property name="link_mass" value="1"/>
-    <xacro:property name="rotor_mass" value="0"/>
-    <!-- NOTE(@nicholasadr): Had to separate independent and dependent joint macro
-                             because urdf will capitalize the first letter of boolean
-                             parameter "true/false" to "True/False", leading to
-                             incorrect joint registration -->
-    <xacro:macro name="independent_joint" params="name parent child">
-        <joint name="${name}" type="revolute" independent="true">
-            <parent link="${parent}"/>
-            <child link="${child}"/>
-            <axis xyz="0 0 1"/>
-            <origin xyz="1.0 0.0 0.0"/>
-            <limit effort="${effort_limit}" velocity="${velocity_limit}"
-                   lower="${joint_lower_limit}" upper="${joint_upper_limit}"/>
-        </joint>
-    </xacro:macro>
-    <xacro:macro name="dependent_joint" params="name parent child">
-        <joint name="${name}" type="revolute" independent="false">
-            <parent link="${parent}"/>
-            <child link="${child}"/>
-            <axis xyz="0 0 1"/>
-            <origin xyz="1.0 0.0 0.0"/>
-            <limit effort="${effort_limit}" velocity="${velocity_limit}"
-                   lower="${joint_lower_limit}" upper="${joint_upper_limit}"/>
-        </joint>
-    </xacro:macro>
-    <xacro:macro name="link" params="name">
-        <link name="${name}">
-            <inertial>
-                <mass value="${link_mass}"/>
-                <origin rpy="0 0 0" xyz="0.5 0 0"/>
-                <inertia ixx="1" ixy="0" ixz="0" iyy="1" iyz="0" izz="1"/>
-            </inertial>
-        </link>
-    </xacro:macro>
-    <xacro:macro name="rotor" params="name">
-        <link name="${name}">
-            <inertial>
-                <mass value="${rotor_mass}"/>
-                <origin rpy="0 0 0" xyz="0 0 0"/>
-                <inertia ixx="1e-4" ixy="0" ixz="0" iyy="1e-4" iyz="0" izz="1e-4"/>
-            </inertial>
-        </link>
-    </xacro:macro>
-    <xacro:macro name="transmission" params="name predecessor successor">
-        <constraint name="${name}" type="rolling">
-            <predecessor link="${predecessor}"/>
-            <successor link="${successor}"/>
-            <ratio value="6.0"/>
-        </constraint>
-    </xacro:macro>
-    <xacro:macro name="base_chain">
-        <xacro:independent_joint name="base_to_link_1" parent="base" child="link_1"/>
-        <xacro:link name="link_1"/>
-        <xacro:dependent_joint name="base_to_rotor_1" parent="base" child="rotor_1"/>
-        <xacro:rotor name="rotor_1"/>
-        <xacro:transmission name="transmission_1" predecessor="link_1" successor="rotor_1"/>
-    </xacro:macro>
-    <xacro:macro name="revolute_rotor_loop" params="idx">
-        <xacro:if value="${idx - 1}">
-            <xacro:independent_joint name="link_${idx - 1}_to_link_${idx}" parent="link_${idx - 1}" child="link_${idx}"/>
-            <xacro:link name="link_${idx}"/>
-            <xacro:dependent_joint name="link_${idx - 1}_to_rotor_${idx}" parent="link_${idx - 1}" child="rotor_${idx}"/>
-            <xacro:rotor name="rotor_${idx}"/>
-            <xacro:transmission name="transmission_${idx}" predecessor="link_${idx}" successor="rotor_${idx}"/>
-            <xacro:revolute_rotor_loop idx="${idx - 1}"/>
-        </xacro:if>
-    </xacro:macro>
+    <xacro:include filename="revolute_rotor_properties.xacro"/>
     <link name="base"/>
-    <xacro:base_chain/>
-    <xacro:revolute_rotor_loop idx="${loop_count}"/>
+    <xacro:root_branch branch_count="1"/>
+    <xacro:serial_chain start_link_idx="1" count="${loop_count - 1}"/>
 </robot>

File: robot-models/revolute_rotor_parallel.xacro (robot description, xacro)
@@ -3,66 +3,5 @@
     <xacro:arg name="loop_count" default="3"/>
     <xacro:property name="loop_count" value="$(arg loop_count)"/>
-    <xacro:property name="effort_limit" value="30"/>
-    <xacro:property name="velocity_limit" value="1."/>
-    <xacro:property name="joint_lower_limit" value="-10"/>
-    <xacro:property name="joint_upper_limit" value="10"/>
-    <xacro:property name="link_mass" value="0.1"/>
-    <xacro:property name="rotor_mass" value="0.05"/>
-    <!-- NOTE(@nicholasadr): Had to separate independent and dependent joint macro
-                             because urdf will capitalize the first letter of boolean
-                             parameter "true/false" to "True/False", leading to
-                             incorrect joint registration -->
-    <xacro:macro name="independent_joint" params="name parent child">
-        <joint name="${name}" type="revolute" independent="true">
-            <parent link="${parent}"/>
-            <child link="${child}"/>
-            <axis xyz="0 0 1"/>
-            <origin xyz="1.0 0.0 0.0"/>
-            <limit effort="${effort_limit}" velocity="${velocity_limit}"
-                   lower="${joint_lower_limit}" upper="${joint_upper_limit}"/>
-        </joint>
-    </xacro:macro>
-    <xacro:macro name="dependent_joint" params="name parent child">
-        <joint name="${name}" type="revolute" independent="false">
-            <parent link="${parent}"/>
-            <child link="${child}"/>
-            <axis xyz="0 0 1"/>
-            <origin xyz="1.0 0.0 0.0"/>
-            <limit effort="${effort_limit}" velocity="${velocity_limit}"
-                   lower="${joint_lower_limit}" upper="${joint_upper_limit}"/>
-        </joint>
-    </xacro:macro>
-    <xacro:macro name="link" params="name">
-        <link name="${name}">
-            <inertial>
-                <mass value="${link_mass}"/>
-                <origin rpy="0 0 0" xyz="0.5 0 0"/>
-                <inertia ixx="1" ixy="0" ixz="0" iyy="1" iyz="0" izz="1"/>
-            </inertial>
-        </link>
-    </xacro:macro>
-    <xacro:macro name="rotor" params="name">
-        <link name="${name}">
-            <inertial>
-                <mass value="${rotor_mass}"/>
-                <origin rpy="0 0 0" xyz="0 0 0"/>
-                <inertia ixx="1e-4" ixy="0" ixz="0" iyy="1e-4" iyz="0" izz="1e-4"/>
-            </inertial>
-        </link>
-    </xacro:macro>
-    <xacro:macro name="transmission" params="name predecessor successor">
-        <constraint name="${name}" type="rolling">
-            <predecessor link="${predecessor}"/>
-            <successor link="${successor}"/>
-            <ratio value="6.0"/>
-        </constraint>
-    </xacro:macro>
-    <xacro:macro name="base_chain">
-        <xacro:independent_joint name="base_to_link_1" parent="base" child="link_1"/>
-        <xacro:link name="link_1"/>
-        <xacro:dependent_joint name="base_to_rotor_1" parent="base" child="rotor_1"/>
-        <xacro:rotor name="rotor_1"/>
-        <xacro:transmission name="transmission_1" predecessor="link_1" successor="rotor_1"/>
-    </xacro:macro>
+    <xacro:include filename="revolute_rotor_properties.xacro"/>
     <xacro:macro name="revolute_rotor_loop" params="idx">
         <xacro:if value="${idx - 1}">
@@ -76,5 +15,5 @@
     </xacro:macro>
     <link name="base"/>
-    <xacro:base_chain/>
+    <xacro:root_branch branch_count="1"/>
     <xacro:revolute_rotor_loop idx="${loop_count}"/>
 </robot>

Commit message: Modify revolute rotor properties

File: robot-models/revolute_rotor_chain.xacro (robot description, xacro)
@@ -6,4 +6,4 @@
     <link name="base"/>
     <xacro:root_branch branch_count="1"/>
-    <xacro:serial_chain start_link_idx="1" count="${loop_count - 1}"/>
+    <xacro:sequential_serial_chain parent_link_idx="1" count="${loop_count}"/>
 </robot>

File: robot-models/revolute_rotor_properties.xacro (robot description, xacro)
@@ -69,17 +69,24 @@
         </xacro:if>
     </xacro:macro>
-    <xacro:macro name="serial_chain" params="start_link_idx count">
-        <xacro:if value="${count}">
-            <xacro:independent_joint name="link_${start_link_idx}_to_link_${start_link_idx + 1}"
-                                     parent="link_${start_link_idx}" child="link_${start_link_idx + 1}"/>
-            <xacro:link name="link_${start_link_idx + 1}"/>
-            <xacro:dependent_joint name="link_${start_link_idx}_to_rotor_${start_link_idx + 1}"
-                                     parent="link_${start_link_idx}" child="rotor_${start_link_idx + 1}"/>
-            <xacro:rotor name="rotor_${start_link_idx+1}"/>
-            <xacro:transmission name="transmission_${start_link_idx + 1}"
-                                predecessor="link_${start_link_idx + 1}"
-                                successor="rotor_${start_link_idx + 1}"/>
-            <xacro:serial_chain start_link_idx="${start_link_idx + 1}" count="${count - 1}"/>
+    <xacro:macro name="one_serial_chain" params="parent_link_idx child_link_idx">
+        <xacro:independent_joint name="link_${parent_link_idx}_to_link_${child_link_idx}"
+                                 parent="link_${parent_link_idx}" child="link_${child_link_idx}"/>
+        <xacro:link name="link_${child_link_idx}"/>
+        <xacro:dependent_joint name="link_${parent_link_idx}_to_rotor_${child_link_idx}"
+                               parent="link_${parent_link_idx}" child="rotor_${child_link_idx}"/>
+        <xacro:rotor name="rotor_${child_link_idx}"/>
+        <xacro:transmission name="transmission_${child_link_idx}"
+                            predecessor="link_${child_link_idx}"
+                            successor="rotor_${child_link_idx}"/>
+    </xacro:macro>
+    <xacro:macro name="sequential_serial_chain" params="parent_link_idx count">
+        <xacro:if value="${count - 1}">
+            <xacro:one_serial_chain parent_link_idx="${parent_link_idx}" child_link_idx="${parent_link_idx + 1}"/>
+            <xacro:sequential_serial_chain parent_link_idx="${parent_link_idx + 1}" count="${count - 1}"/>
         </xacro:if>
     </xacro:macro>
+    <xacro:macro name="nonsequential_serial_chain" params="parent_link_idx first_child_link_idx count">
+        <xacro:one_serial_chain parent_link_idx="${parent_link_idx}" child_link_idx="${first_child_link_idx}"/>
+        <xacro:sequential_serial_chain parent_link_idx="${first_child_link_idx}" count="${count - 1}"/>
+    </xacro:macro>
 </robot>
