Commit message: Actually fix urdf now - match cheetah-software convention

File: robot-models/mini_cheetah_properties.xacro (robot description, xacro)
@@ -92,7 +92,7 @@
                 <mass value="0.064"/>
                 <origin xyz="0.0 0.0 -0.061"/>
-                <inertia ixx="${245 * 1e-6}" ixy="0.0"
+                <inertia ixx="${6 * 1e-6}" ixy="0.0"
                          ixz="0.0" iyy="${248 * 1e-6}"
-                         iyz="0.0" izz="${6 * 1e-6}"/>
+                         iyz="0.0" izz="${245 * 1e-6}"/>
             </inertial>
             <!-- TODO(@MatthewChignoli): Do collision and visual stuff later -->

Commit message: WIP

File: robot-models/mini_cheetah_properties.xacro (robot description, xacro)
@@ -35,9 +35,9 @@
             </inertial>
         </link>
-        <constraint name="${prefix}_abad_tranmission" type="rolling">
-            <predecessor link="${prefix}_abad_link"/>
-            <successor link="${prefix}_abad_rotor"/>
-            <ratio value="6.0"/>
-        </constraint>
+        <joint_constraint name="${prefix}_abad_tranmission">
+            <parent link="${prefix}_abad_link"/>
+            <child link="${prefix}_abad_rotor"/>
+            <gear_ratio value="6.0"/>
+        </joint_constraint>
     </xacro:macro>
     <!-- Hip Macro -->
@@ -74,9 +74,9 @@
             </inertial>
         </link>
-        <constraint name="${prefix}_hip_tranmission" type="rolling">
-            <predecessor link="${prefix}_hip_link"/>
-            <successor link="${prefix}_hip_rotor"/>
-            <ratio value="6.0"/>
-        </constraint>
+        <joint_constraint name="${prefix}_hip_tranmission">
+            <parent link="${prefix}_hip_link"/>
+            <child link="${prefix}_hip_rotor"/>
+            <gear_ratio value="6.0"/>
+        </joint_constraint>
     </xacro:macro>
     <!-- Knee Macro -->
@@ -112,9 +112,9 @@
             </inertial>
         </link>
-        <constraint name="${prefix}_knee_tranmission" type="rolling">
-            <predecessor link="${prefix}_knee_link"/>
-            <successor link="${prefix}_knee_rotor"/>
-            <ratio value="9.33"/>
-        </constraint>
+        <joint_constraint name="${prefix}_knee_tranmission">
+            <parent link="${prefix}_knee_link"/>
+            <child link="${prefix}_knee_rotor"/>
+            <gear_ratio value="9.33"/>
+        </joint_constraint>
     </xacro:macro>
 </robot>

File: robot-models/mit_humanoid.xacro (robot description, xacro)
@@ -33,7 +33,7 @@
         </link>
         <constraint name="${prefix}hipz_transmission" type="rolling">
-            <predecessor link="${prefix}hip_rz_link"/>
-            <successor link="${prefix}hip_rz_rotor"/>
-            <ratio value="6.0"/>
+            <parent link="${prefix}hip_rz_link"/>
+            <child link="${prefix}hip_rz_rotor"/>
+            <gear_ratio value="6.0"/>
         </constraint>
     </xacro:macro>
@@ -69,9 +69,9 @@
             </inertial>
         </link>
-        <constraint name="${prefix}hipx_transmission" type="rolling">
-            <predecessor link="${prefix}hip_rx_link"/>
-            <successor link="${prefix}hip_rx_rotor"/>
-            <ratio value="6.0"/>
-        </constraint>
+        <joint_constraint name="${prefix}hipx_transmission">
+            <parent link="${prefix}hip_rx_link"/>
+            <child link="${prefix}hip_rx_rotor"/>
+            <gear_ratio value="6.0"/>
+        </joint_constraint>
     </xacro:macro>
     <!-- Hip Flexion/Extension -->
@@ -105,9 +105,9 @@
             </inertial>
         </link>
-        <constraint name="${prefix}hipy_transmission" type="rolling">
-            <predecessor link="${prefix}hip_ry_link"/>
-            <successor link="${prefix}hip_ry_rotor"/>
-            <ratio value="6.0"/>
-        </constraint>
+        <joint_constraint name="${prefix}hipy_transmission">
+            <parent link="${prefix}hip_ry_link"/>
+            <child link="${prefix}hip_ry_rotor"/>
+            <gear_ratio value="6.0"/>
+        </joint_constraint>
     </xacro:macro>
     <!-- Knee Flexion/Extension -->
@@ -141,9 +141,9 @@
             </inertial>
         </link>
-        <constraint name="${prefix}knee_transmission" type="rolling">
-            <predecessor link="${prefix}knee_link"/>
-            <successor link="${prefix}knee_rotor"/>
-            <ratio value="12.0"/>
-        </constraint>
+        <joint_constraint name="${prefix}knee_transmission">
+            <parent link="${prefix}knee_link"/>
+            <child link="${prefix}knee_rotor"/>
+            <gear_ratio value="12.0"/>
+        </joint_constraint>
     </xacro:macro>
     <!-- Ankle Flexion/Extension -->
@@ -177,9 +177,9 @@
             </inertial>
         </link>
-        <constraint name="${prefix}ankle_transmission" type="rolling">
-            <predecessor link="${prefix}ankle_link"/>
-            <successor link="${prefix}ankle_rotor"/>
-            <ratio value="12.0"/>
-        </constraint>
+        <joint_constraint name="${prefix}ankle_transmission">
+            <parent link="${prefix}ankle_link"/>
+            <child link="${prefix}ankle_rotor"/>
+            <gear_ratio value="12.0"/>
+        </joint_constraint>
     </xacro:macro>
     <!-- Shoulder Y-axis -->
@@ -213,9 +213,9 @@
             </inertial>
         </link>
-        <constraint name="${prefix}shouldery_transmission" type="rolling">
-            <predecessor link="${prefix}shoulder_ry_link"/>
-            <successor link="${prefix}shoulder_ry_rotor"/>
-            <ratio value="6.0"/>
-        </constraint>
+        <joint_constraint name="${prefix}shouldery_transmission">
+            <parent link="${prefix}shoulder_ry_link"/>
+            <child link="${prefix}shoulder_ry_rotor"/>
+            <gear_ratio value="6.0"/>
+        </joint_constraint>
     </xacro:macro>
     <!-- Shoulder X-axis -->
@@ -249,9 +249,9 @@
             </inertial>
         </link>
-        <constraint name="${prefix}shoulderx_transmission" type="rolling">
-            <predecessor link="${prefix}shoulder_rx_link"/>
-            <successor link="${prefix}shoulder_rx_rotor"/>
-            <ratio value="6.0"/>
-        </constraint>
+        <joint_constraint name="${prefix}shoulderx_transmission">
+            <parent link="${prefix}shoulder_rx_link"/>
+            <child link="${prefix}shoulder_rx_rotor"/>
+            <gear_ratio value="6.0"/>
+        </joint_constraint>
     </xacro:macro>
     <!-- Shoulder Z-axis -->
@@ -285,9 +285,9 @@
             </inertial>
         </link>
-        <constraint name="${prefix}shoulderz_transmission" type="rolling">
-            <predecessor link="${prefix}shoulder_rz_link"/>
-            <successor link="${prefix}shoulder_rz_rotor"/>
-            <ratio value="6.0"/>
-        </constraint>
+        <joint_constraint name="${prefix}shoulderz_transmission">
+            <parent link="${prefix}shoulder_rz_link"/>
+            <child link="${prefix}shoulder_rz_rotor"/>
+            <gear_ratio value="6.0"/>
+        </joint_constraint>
     </xacro:macro>
     <!-- Elbow Flexion/Extension -->
@@ -321,9 +321,9 @@
             </inertial>
         </link>
-        <constraint name="${prefix}elbow_transmission" type="rolling">
-            <predecessor link="${prefix}elbow_link"/>
-            <successor link="${prefix}elbow_rotor"/>
-            <ratio value="9.0"/>
-        </constraint>
+        <joint_constraint name="${prefix}elbow_transmission">
+            <parent link="${prefix}elbow_link"/>
+            <child link="${prefix}elbow_rotor"/>
+            <gear_ratio value="9.0"/>
+        </joint_constraint>
     </xacro:macro>
     <!-- End of macro definitions -->

File: robot-models/mit_humanoid_leg.xacro (robot description, xacro)
@@ -32,9 +32,9 @@
             </inertial>
         </link>
-        <constraint name="hipz_transmission" type="rolling">
-            <predecessor link="${prefix}hip_rz_link"/>
-            <successor link="${prefix}hip_rz_rotor"/>
-            <ratio value="6.0"/>
-        </constraint>
+        <joint_constraint name="hipz_transmission">
+            <parent link="${prefix}hip_rz_link"/>
+            <child link="${prefix}hip_rz_rotor"/>
+            <gear_ratio value="6.0"/>
+        </joint_constraint>
     </xacro:macro>
     <!-- Hip Abduction/Adduction -->
@@ -69,9 +69,9 @@
             </inertial>
         </link>
-        <constraint name="hipx_transmission" type="rolling">
-            <predecessor link="${prefix}hip_rx_link"/>
-            <successor link="${prefix}hip_rx_rotor"/>
-            <ratio value="6.0"/>
-        </constraint>
+        <joint_constraint name="hipx_transmission">
+            <parent link="${prefix}hip_rx_link"/>
+            <child link="${prefix}hip_rx_rotor"/>
+            <gear_ratio value="6.0"/>
+        </joint_constraint>
     </xacro:macro>
     <!-- Hip Flexion/Extension -->
@@ -105,9 +105,9 @@
             </inertial>
         </link>
-        <constraint name="hipy_transmission" type="rolling">
-            <predecessor link="${prefix}hip_ry_link"/>
-            <successor link="${prefix}hip_ry_rotor"/>
-            <ratio value="6.0"/>
-        </constraint>
+        <joint_constraint name="hipy_transmission">
+            <parent link="${prefix}hip_ry_link"/>
+            <child link="${prefix}hip_ry_rotor"/>
+            <gear_ratio value="6.0"/>
+        </joint_constraint>
     </xacro:macro>
     <!-- Knee Flexion/Extension -->
@@ -141,9 +141,9 @@
             </inertial>
         </link>
-        <constraint name="knee_transmission" type="rolling">
-            <predecessor link="${prefix}knee_link"/>
-            <successor link="${prefix}knee_rotor"/>
-            <ratio value="12.0"/>
-        </constraint>
+        <joint_constraint name="knee_transmission">
+            <parent link="${prefix}knee_link"/>
+            <child link="${prefix}knee_rotor"/>
+            <gear_ratio value="12.0"/>
+        </joint_constraint>
     </xacro:macro>
     <!-- Ankle Flexion/Extension -->
@@ -177,9 +177,9 @@
             </inertial>
         </link>
-        <constraint name="ankle_transmission" type="rolling">
-            <predecessor link="${prefix}ankle_link"/>
-            <successor link="${prefix}ankle_rotor"/>
-            <ratio value="12.0"/>
-        </constraint>
+        <joint_constraint name="ankle_transmission">
+            <parent link="${prefix}ankle_link"/>
+            <child link="${prefix}ankle_rotor"/>
+            <gear_ratio value="12.0"/>
+        </joint_constraint>
     </xacro:macro>
     <link name="base"/>

Commit message: Approximate system benchmark

File: robot-models/mini_cheetah_properties.xacro (robot description, xacro)
@@ -49,4 +49,23 @@
         </constraint>
     </xacro:macro>
+    <xacro:macro name="abad_approx" params="prefix x_sign y_sign">
+        <joint name="torso_to_${prefix}_abad_j" type="revolute">
+            <axis xyz="1 0 0"/>
+            <origin xyz="${x_sign * 0.19} ${y_sign * 0.049} 0.0"/>
+            <parent link="Floating Base"/>
+            <child link="${prefix}_abad_link"/>
+            <limit effort="${effort_limit}" velocity="${velocity_limit}"
+                   lower="${joint_lower_limit}" upper="${joint_upper_limit}"/>
+        </joint>
+        <link name="${prefix}_abad_link">
+            <inertial>
+                <mass value="0.54"/>
+                <origin xyz="0.0 ${y_sign * 0.036} 0."/>
+                <inertia ixx="${381 * 1e-6}" ixy="${y_sign * 58 * 1e-6}"
+                         ixz="${0.45 * 1e-6}" iyy="${560 * 1e-6}"
+                         iyz="${y_sign * .95 * 1e-6}" izz="${444 * 1e-6}"/>
+            </inertial>
+        </link>
+    </xacro:macro>
     <!-- Hip Macro -->
     <xacro:macro name="hip" params="prefix x_sign y_sign">
@@ -92,4 +111,23 @@
         </constraint>
     </xacro:macro>
+    <xacro:macro name="hip_approx" params="prefix x_sign y_sign">
+        <joint name="${prefix}_abad_to_hip_j" type="revolute">
+            <axis xyz="0 1 0"/>
+            <origin xyz="0 ${y_sign * 0.062} 0.0" rpy="0 0 ${pi}"/>
+            <parent link="${prefix}_abad_link"/>
+            <child link="${prefix}_hip_link"/>
+            <limit effort="${effort_limit}" velocity="${velocity_limit}"
+                   lower="${joint_lower_limit}" upper="${joint_upper_limit}"/>
+        </joint>
+        <link name="${prefix}_hip_link">
+            <inertial>
+                <mass value="0.634"/>
+                <origin xyz="0.0 ${y_sign * 0.016} -0.02"/>
+                <inertia ixx="${1983 * 1e-6}" ixy="${y_sign * 245 * 1e-6}"
+                         ixz="${13 * 1e-6}" iyy="${2103 * 1e-6}"
+                         iyz="${y_sign * 1.5 * 1e-6}" izz="${408 * 1e-6}"/>
+            </inertial>
+        </link>
+    </xacro:macro>
     <!-- Knee Macro -->
     <xacro:macro name="knee" params="prefix x_sign y_sign">
@@ -134,3 +172,22 @@
         </constraint>
     </xacro:macro>
+    <xacro:macro name="knee_approx" params="prefix x_sign y_sign">
+        <joint name="${prefix}_hip_to_knee_j" type="revolute">
+            <axis xyz="0 1 0"/>
+            <origin xyz="0.0 0.0 -0.209"/>
+            <parent link="${prefix}_hip_link"/>
+            <child link="${prefix}_knee_link"/>
+            <limit effort="${effort_limit}" velocity="${velocity_limit}"
+                   lower="${joint_lower_limit}" upper="${joint_upper_limit}"/>
+        </joint>
+        <link name="${prefix}_knee_link">
+            <inertial>
+                <mass value="0.064"/>
+                <origin xyz="0.0 0.0 -0.061"/>
+                <inertia ixx="${6 * 1e-6}" ixy="0.0"
+                         ixz="0.0" iyy="${248 * 1e-6}"
+                         iyz="0.0" izz="${245 * 1e-6}"/>
+            </inertial>
+        </link>
+    </xacro:macro>
 </robot>
