Commit message: WIP pinocchio forward dynamics to include Tello Knee-Ankle Differentials:
- increase error margin
- add Tello Knee-Ankle Differentials in Cluster Tree Model and urdf
- fix Tello Hip Differentials urdf
- add joint names to MiniCheetah, RevoluteChainWithRotor, RevoluteChainWithAndWithoutRotor

File: robot-models/tello_leg.urdf (robot description, URDF)
Before this commit: robot tello_leg, 7 links, 6 joints
Links:
- added link right-foot, mass 0.1025
- added link right-knee-ankle-rotor-1, mass 0.07
- added link right-knee-ankle-rotor-2, mass 0.07
- added link right-shin, mass 0.3072
Joints:
- added joint right-shin-to-foot: type revolute, parent right-shin, child right-foot, origin xyz=0.0 0.0 -260e-03 rpy=0.0 0.0 0.0, axis 0 1 0, limit lower=-10 upper=10 effort=150 velocity=100
- added joint right-thigh-to-knee-ankle-rotor-1: type revolute, parent right-thigh, child right-knee-ankle-rotor-1, origin xyz=0.0 26.55e-03 0.0 rpy=-1.5707963 0.0 0.0, axis 0 0 1, limit lower=-10 upper=10 effort=150 velocity=100
- added joint right-thigh-to-knee-ankle-rotor-2: type revolute, parent right-thigh, child right-knee-ankle-rotor-2, origin xyz=0.0 -26.55e-03 0.0 rpy=-1.5707963 0.0 -3.1415927, axis 0 0 1, limit lower=-10 upper=10 effort=150 velocity=100
- added joint right-thigh-to-shin: type revolute, parent right-thigh, child right-shin, origin xyz=0.0 0.0 -226.8e-03 rpy=0.0 0.0 0.0, axis 0 1 0, limit lower=-10 upper=10 effort=150 velocity=100
