Commit message: Fixes to tello:
- fix joint rpy
- change arm sequence to left,right for consistency
- add separate left,right arm link inertia
- add separate left,right arm link origin

File: robot-models/tello_humanoid.urdf (robot description, URDF)
Before this commit: robot tello_humanoid, 37 links, 36 joints
Links:
- removed link base
- added link ground, mass 2.3008
Joints:
- removed joint base-to-left-hip-clamp
- removed joint base-to-left-hip-clamp-rotor
- removed joint base-to-left-shoulder-ry
- removed joint base-to-left-shoulder-ry-rotor
- removed joint base-to-right-hip-clamp
- removed joint base-to-right-hip-clamp-rotor
- removed joint base-to-right-shoulder-ry
- removed joint base-to-right-shoulder-ry-rotor
- removed joint left-shoulder-rx-to-left-shoulder-rz
- removed joint left-shoulder-rx-to-left-shoulder-rz-rotor
- removed joint left-shoulder-ry-to-left-shoulder-rx
- removed joint left-shoulder-ry-to-left-shoulder-rx-rotor
- removed joint left-shoulder-rz-to-left-elbow
- removed joint left-shoulder-rz-to-left-elbow-rotor
- removed joint right-shoulder-rx-to-right-shoulder-rz
- removed joint right-shoulder-rx-to-right-shoulder-rz-rotor
- removed joint right-shoulder-ry-to-right-shoulder-rx
- removed joint right-shoulder-ry-to-right-shoulder-rx-rotor
- removed joint right-shoulder-rz-to-right-elbow
- removed joint right-shoulder-rz-to-right-elbow-rotor
- added joint ground-to-left-hip-clamp: type revolute, parent ground, child left-hip-clamp, origin xyz=0.0 126e-03 -87e-03 rpy=0.0 0.0 0.0, axis 0 0 1, limit lower=-10 upper=10 effort=150 velocity=100
- added joint ground-to-left-hip-clamp-rotor: type revolute, parent ground, child left-hip-clamp-rotor, origin xyz=0.0 126e-03 -26e-03 rpy=3.1415927 0.0 0.0, axis 0 0 1, limit lower=-10 upper=10 effort=150 velocity=100
- added joint ground-to-left-shoulder-ry: type revolute, parent ground, child left-shoulder-ry, origin xyz=0.01346 0.17608 0.24657 rpy=0.0 0.0 0.0, axis 0 1 0, limit lower=-10 upper=10 effort=150 velocity=100
- added joint ground-to-left-shoulder-ry-rotor: type revolute, parent ground, child left-shoulder-ry-rotor, origin xyz=0.01346 0.16 0.24657 rpy=0.0 0.0 0.0, axis 0 1 0, limit lower=-10 upper=10 effort=150 velocity=100
- added joint ground-to-right-hip-clamp: type revolute, parent ground, child right-hip-clamp, origin xyz=0.0 -126e-03 -87e-03 rpy=0.0 0.0 0.0, axis 0 0 1, limit lower=-10 upper=10 effort=150 velocity=100
- added joint ground-to-right-hip-clamp-rotor: type revolute, parent ground, child right-hip-clamp-rotor, origin xyz=0.0 -126e-03 -26e-03 rpy=0.0 0.0 0.0, axis 0 0 1, limit lower=-10 upper=10 effort=150 velocity=100
- added joint ground-to-right-shoulder-ry: type revolute, parent ground, child right-shoulder-ry, origin xyz=0.01346 -0.17608 0.24657 rpy=0.0 0.0 0.0, axis 0 1 0, limit lower=-10 upper=10 effort=150 velocity=100
- added joint ground-to-right-shoulder-ry-rotor: type revolute, parent ground, child right-shoulder-ry-rotor, origin xyz=0.01346 -0.16 0.24657 rpy=0.0 0.0 0.0, axis 0 1 0, limit lower=-10 upper=10 effort=150 velocity=100
- added joint left-shoulder-rx-to-shoulder-rz: type revolute, parent left-shoulder-rx, child left-shoulder-rz, origin xyz=0.0 0.0 -0.1025 rpy=0.0 0.0 0.0, axis 0 0 1, limit lower=-10 upper=10 effort=150 velocity=100
- added joint left-shoulder-rx-to-shoulder-rz-rotor: type revolute, parent left-shoulder-rx, child left-shoulder-rz-rotor, origin xyz=0.0 0.0 -0.1025 rpy=0.0 0.0 0.0, axis 0 0 1, limit lower=-10 upper=10 effort=150 velocity=100
- added joint left-shoulder-ry-to-shoulder-rx: type revolute, parent left-shoulder-ry, child left-shoulder-rx, origin xyz=0.0 0.0575 0.0 rpy=0.0 0.0 0.0, axis 1 0 0, limit lower=-10 upper=10 effort=150 velocity=100
- added joint left-shoulder-ry-to-shoulder-rx-rotor: type revolute, parent left-shoulder-ry, child left-shoulder-rx-rotor, origin xyz=0.0 0.0575 0.0 rpy=0.0 0.0 0.0, axis 1 0 0, limit lower=-10 upper=10 effort=150 velocity=100
- added joint left-shoulder-rz-to-elbow: type revolute, parent left-shoulder-rz, child left-elbow, origin xyz=0.0 0.0 -0.1455 rpy=0.0 0.0 0.0, axis 0 1 0, limit lower=-10 upper=10 effort=150 velocity=100
- added joint left-shoulder-rz-to-elbow-rotor: type revolute, parent left-shoulder-rz, child left-elbow-rotor, origin xyz=0.0 -0.0325 -0.06 rpy=0.0 0.0 0.0, axis 0 1 0, limit lower=-10 upper=10 effort=150 velocity=100
- added joint right-shoulder-rx-to-shoulder-rz: type revolute, parent right-shoulder-rx, child right-shoulder-rz, origin xyz=0.0 0.0 -0.1025 rpy=0.0 0.0 0.0, axis 0 0 1, limit lower=-10 upper=10 effort=150 velocity=100
- added joint right-shoulder-rx-to-shoulder-rz-rotor: type revolute, parent right-shoulder-rx, child right-shoulder-rz-rotor, origin xyz=0.0 0.0 -0.1025 rpy=0.0 0.0 0.0, axis 0 0 1, limit lower=-10 upper=10 effort=150 velocity=100
- added joint right-shoulder-ry-to-shoulder-rx: type revolute, parent right-shoulder-ry, child right-shoulder-rx, origin xyz=0.0 -0.0575 0.0 rpy=0.0 0.0 0.0, axis 1 0 0, limit lower=-10 upper=10 effort=150 velocity=100
- added joint right-shoulder-ry-to-shoulder-rx-rotor: type revolute, parent right-shoulder-ry, child right-shoulder-rx-rotor, origin xyz=0.0 -0.0575 0.0 rpy=0.0 0.0 0.0, axis 1 0 0, limit lower=-10 upper=10 effort=150 velocity=100
- added joint right-shoulder-rz-to-elbow: type revolute, parent right-shoulder-rz, child right-elbow, origin xyz=0.0 0.0 -0.1455 rpy=0.0 0.0 0.0, axis 0 1 0, limit lower=-10 upper=10 effort=150 velocity=100
- added joint right-shoulder-rz-to-elbow-rotor: type revolute, parent right-shoulder-rz, child right-elbow-rotor, origin xyz=0.0 0.0325 -0.06 rpy=0.0 0.0 0.0, axis 0 1 0, limit lower=-10 upper=10 effort=150 velocity=100
- joint left-hip-clamp-to-hip-rotor-1: origin xyz=0.0 0.04 0.0 rpy=-1.5707963 0.0 -3.1415927 -> xyz=0.0 0.04 0.0 rpy=-1.5707963 3.1415927 0.0
- joint left-hip-clamp-to-hip-rotor-2: origin xyz=0.0 -0.04 0.0 rpy=-1.5707963 0.0 0.0 -> xyz=0.0 -0.04 0.0 rpy=1.5707963 0.0 0.0
- joint left-thigh-to-knee-ankle-rotor-1: origin xyz=0.0 26.55e-03 0.0 rpy=-1.5707963 0.0 0.0 -> xyz=0.0 26.55e-03 0.0 rpy=1.5707963 0.0 0.0
- joint left-thigh-to-knee-ankle-rotor-2: origin xyz=0.0 -26.55e-03 0.0 rpy=-1.5707963 0.0 -3.1415927 -> xyz=0.0 -26.55e-03 0.0 rpy=-1.5707963 3.1415927 0.0
- joint right-hip-clamp-to-hip-rotor-1: origin xyz=0.0 0.04 0.0 rpy=-1.5707963 0.0 -3.1415927 -> xyz=0.0 0.04 0.0 rpy=-1.5707963 3.1415927 0.0
- joint right-hip-clamp-to-hip-rotor-2: origin xyz=0.0 -0.04 0.0 rpy=-1.5707963 0.0 0.0 -> xyz=0.0 -0.04 0.0 rpy=1.5707963 0.0 0.0
- joint right-thigh-to-knee-ankle-rotor-1: origin xyz=0.0 26.55e-03 0.0 rpy=-1.5707963 0.0 0.0 -> xyz=0.0 26.55e-03 0.0 rpy=1.5707963 0.0 0.0
- joint right-thigh-to-knee-ankle-rotor-2: origin xyz=0.0 -26.55e-03 0.0 rpy=-1.5707963 0.0 -3.1415927 -> xyz=0.0 -26.55e-03 0.0 rpy=-1.5707963 3.1415927 0.0

File: robot-models/tello_humanoid.xacro (robot description, xacro)
@@ -2,11 +2,11 @@
 <robot name="tello_humanoid" xmlns:xacro="http://ros.org/wiki/xacro">
     <xacro:include filename="tello_properties.xacro"/>
-    <xacro:property name="base" value="base"/>
+    <xacro:property name="base" value="ground"/>
     <!-- Torso -->
     <xacro:torso name="${base}"/>
     <!-- Left Hip Cluster -->
-    <xacro:L_independent_hip_clamp_rotor_joint parent="${base}"/>
+    <xacro:L_dependent_hip_clamp_rotor_joint parent="${base}"/>
     <xacro:hip_clamp_rotor prefix="left-"/>
-    <xacro:L_dependent_hip_clamp_joint parent="${base}"/>
+    <xacro:L_independent_hip_clamp_joint parent="${base}"/>
     <xacro:hip_clamp prefix="left-"/>
     <!-- Left Hip Differentials -->
@@ -29,7 +29,7 @@
     <xacro:foot prefix="left-"/>
     <!-- Right Hip Cluster -->
-    <xacro:R_independent_hip_clamp_rotor_joint parent="${base}"/>
+    <xacro:R_dependent_hip_clamp_rotor_joint parent="${base}"/>
     <xacro:hip_clamp_rotor prefix="right-"/>
-    <xacro:R_dependent_hip_clamp_joint parent="${base}"/>
+    <xacro:R_independent_hip_clamp_joint parent="${base}"/>
     <xacro:hip_clamp prefix="right-"/>
     <!-- Right Hip Differentials -->
@@ -52,42 +52,42 @@
     <xacro:foot prefix="right-"/>
     <!-- Left Shoulder RY -->
-    <xacro:L_independent_shoulder_ry_rotor_joint parent="${base}"/>
+    <xacro:L_independent_shoulder_ry_joint parent="${base}"/>
+    <xacro:left_shoulder_ry/>
+    <xacro:L_dependent_shoulder_ry_rotor_joint parent="${base}"/>
     <xacro:shoulder_ry_rotor prefix="left-"/>
-    <xacro:L_dependent_shoulder_ry_joint parent="${base}"/>
-    <xacro:shoulder_ry prefix="left-"/>
     <!-- Left Shoulder RX -->
-    <xacro:L_independent_shoulder_rx_rotor_joint parent="left-shoulder-ry"/>
+    <xacro:L_independent_shoulder_rx_joint parent="left-shoulder-ry"/>
+    <xacro:left_shoulder_rx/>
+    <xacro:L_dependent_shoulder_rx_rotor_joint parent="left-shoulder-ry"/>
     <xacro:shoulder_rx_rotor prefix="left-"/>
-    <xacro:L_dependent_shoulder_rx_joint parent="left-shoulder-ry"/>
-    <xacro:shoulder_rx prefix="left-"/>
     <!-- Left Shoulder RZ -->
-    <xacro:L_independent_shoulder_rz_rotor_joint parent="left-shoulder-rx"/>
+    <xacro:L_independent_shoulder_rz_joint parent="left-shoulder-rx"/>
+    <xacro:left_shoulder_rz/>
+    <xacro:L_dependent_shoulder_rz_rotor_joint parent="left-shoulder-rx"/>
     <xacro:shoulder_rz_rotor prefix="left-"/>
-    <xacro:L_dependent_shoulder_rz_joint parent="left-shoulder-rx"/>
-    <xacro:shoulder_rz prefix="left-"/>
     <!-- Left Elbow -->
-    <xacro:L_independent_elbow_rotor_joint parent="left-shoulder-rz"/>
+    <xacro:L_independent_elbow_joint parent="left-shoulder-rz"/>
+    <xacro:left_elbow/>
+    <xacro:L_dependent_elbow_rotor_joint parent="left-shoulder-rz"/>
     <xacro:elbow_rotor prefix="left-"/>
-    <xacro:L_dependent_elbow_joint parent="left-shoulder-rz"/>
-    <xacro:elbow prefix="left-"/>
     <!-- Right Shoulder RY -->
-    <xacro:R_independent_shoulder_ry_rotor_joint parent="${base}"/>
+    <xacro:R_independent_shoulder_ry_joint parent="${base}"/>
+    <xacro:right_shoulder_ry/>
+    <xacro:R_dependent_shoulder_ry_rotor_joint parent="${base}"/>
     <xacro:shoulder_ry_rotor prefix="right-"/>
-    <xacro:R_dependent_shoulder_ry_joint parent="${base}"/>
-    <xacro:shoulder_ry prefix="right-"/>
     <!-- Right Shoulder RX -->
-    <xacro:R_independent_shoulder_rx_rotor_joint parent="right-shoulder-ry"/>
+    <xacro:R_independent_shoulder_rx_joint parent="right-shoulder-ry"/>
+    <xacro:right_shoulder_rx/>
+    <xacro:R_dependent_shoulder_rx_rotor_joint parent="right-shoulder-ry"/>
     <xacro:shoulder_rx_rotor prefix="right-"/>
-    <xacro:R_dependent_shoulder_rx_joint parent="right-shoulder-ry"/>
-    <xacro:shoulder_rx prefix="right-"/>
     <!-- Right Shoulder RZ -->
-    <xacro:R_independent_shoulder_rz_rotor_joint parent="right-shoulder-rx"/>
+    <xacro:R_independent_shoulder_rz_joint parent="right-shoulder-rx"/>
+    <xacro:right_shoulder_rz/>
+    <xacro:R_dependent_shoulder_rz_rotor_joint parent="right-shoulder-rx"/>
     <xacro:shoulder_rz_rotor prefix="right-"/>
-    <xacro:R_dependent_shoulder_rz_joint parent="right-shoulder-rx"/>
-    <xacro:shoulder_rz prefix="right-"/>
     <!-- Right Elbow -->
-    <xacro:R_independent_elbow_rotor_joint parent="right-shoulder-rz"/>
+    <xacro:R_independent_elbow_joint parent="right-shoulder-rz"/>
+    <xacro:right_elbow/>
+    <xacro:R_dependent_elbow_rotor_joint parent="right-shoulder-rz"/>
     <xacro:elbow_rotor prefix="right-"/>
-    <xacro:R_dependent_elbow_joint parent="right-shoulder-rz"/>
-    <xacro:elbow prefix="right-"/>
 </robot>

File: robot-models/tello_humanoid_approximate.urdf (robot description, URDF)
Before this commit: robot tello_humanoid_approximate, 19 links, 18 joints
Joints:
- removed joint left-shoulder-rx-to-left-shoulder-rz
- removed joint left-shoulder-ry-to-left-shoulder-rx
- removed joint left-shoulder-rz-to-left-elbow
- removed joint right-shoulder-rx-to-right-shoulder-rz
- removed joint right-shoulder-ry-to-right-shoulder-rx
- removed joint right-shoulder-rz-to-right-elbow
- added joint left-shoulder-rx-to-shoulder-rz: type revolute, parent left-shoulder-rx, child left-shoulder-rz, origin xyz=0.0 0.0 -0.1025 rpy=0.0 0.0 0.0, axis 0 0 1, limit lower=-10 upper=10 effort=150 velocity=100
- added joint left-shoulder-ry-to-shoulder-rx: type revolute, parent left-shoulder-ry, child left-shoulder-rx, origin xyz=0.0 0.0575 0.0 rpy=0.0 0.0 0.0, axis 1 0 0, limit lower=-10 upper=10 effort=150 velocity=100
- added joint left-shoulder-rz-to-elbow: type revolute, parent left-shoulder-rz, child left-elbow, origin xyz=0.0 0.0 -0.1455 rpy=0.0 0.0 0.0, axis 0 1 0, limit lower=-10 upper=10 effort=150 velocity=100
- added joint right-shoulder-rx-to-shoulder-rz: type revolute, parent right-shoulder-rx, child right-shoulder-rz, origin xyz=0.0 0.0 -0.1025 rpy=0.0 0.0 0.0, axis 0 0 1, limit lower=-10 upper=10 effort=150 velocity=100
- added joint right-shoulder-ry-to-shoulder-rx: type revolute, parent right-shoulder-ry, child right-shoulder-rx, origin xyz=0.0 -0.0575 0.0 rpy=0.0 0.0 0.0, axis 1 0 0, limit lower=-10 upper=10 effort=150 velocity=100
- added joint right-shoulder-rz-to-elbow: type revolute, parent right-shoulder-rz, child right-elbow, origin xyz=0.0 0.0 -0.1455 rpy=0.0 0.0 0.0, axis 0 1 0, limit lower=-10 upper=10 effort=150 velocity=100
- joint base-to-left-shoulder-ry: origin xyz=0.01346 -0.17608 0.24657 rpy=0.0 0.0 0.0 -> xyz=0.01346 0.17608 0.24657 rpy=0.0 0.0 0.0
- joint base-to-right-shoulder-ry: origin xyz=0.01346 0.17608 0.24657 rpy=0.0 0.0 0.0 -> xyz=0.01346 -0.17608 0.24657 rpy=0.0 0.0 0.0

File: robot-models/tello_humanoid_approximate.xacro (robot description, xacro)
@@ -33,25 +33,25 @@
     <!-- Left Shoulder RY -->
     <xacro:L_independent_shoulder_ry_joint parent="${base}"/>
-    <xacro:shoulder_ry prefix="left-"/>
+    <xacro:left_shoulder_ry/>
     <!-- Left Shoulder RX -->
     <xacro:L_independent_shoulder_rx_joint parent="left-shoulder-ry"/>
-    <xacro:shoulder_rx prefix="left-"/>
+    <xacro:left_shoulder_rx/>
     <!-- Left Shoulder RZ -->
     <xacro:L_independent_shoulder_rz_joint parent="left-shoulder-rx"/>
-    <xacro:shoulder_rz prefix="left-"/>
+    <xacro:left_shoulder_rz/>
     <!-- Left Elbow -->
     <xacro:L_independent_elbow_joint parent="left-shoulder-rz"/>
-    <xacro:elbow prefix="left-"/>
+    <xacro:left_elbow/>
     <!-- Right Shoulder RY -->
     <xacro:R_independent_shoulder_ry_joint parent="${base}"/>
-    <xacro:shoulder_ry prefix="right-"/>
+    <xacro:right_shoulder_ry/>
     <!-- Right Shoulder RX -->
     <xacro:R_independent_shoulder_rx_joint parent="right-shoulder-ry"/>
-    <xacro:shoulder_rx prefix="right-"/>
+    <xacro:right_shoulder_rx/>
     <!-- Right Shoulder RZ -->
     <xacro:R_independent_shoulder_rz_joint parent="right-shoulder-rx"/>
-    <xacro:shoulder_rz prefix="right-"/>
+    <xacro:right_shoulder_rz/>
     <!-- Right Elbow -->
     <xacro:R_independent_elbow_joint parent="right-shoulder-rz"/>
-    <xacro:elbow prefix="right-"/>
+    <xacro:right_elbow/>
 </robot>

File: robot-models/tello_legs.urdf (robot description, URDF)
Before this commit: robot tello_legs, 21 links, 20 joints
Joints:
- joint ground-to-left-hip-clamp-rotor: origin xyz=0.0 126e-03 -26e-03 rpy=-3.1415927 0.0 0.0 -> xyz=0.0 126e-03 -26e-03 rpy=3.1415927 0.0 0.0
- joint left-hip-clamp-to-hip-rotor-1: origin xyz=0.0 0.04 0.0 rpy=-1.5707963 0.0 -3.1415927 -> xyz=0.0 0.04 0.0 rpy=-1.5707963 3.1415927 0.0
- joint left-hip-clamp-to-hip-rotor-2: origin xyz=0.0 -0.04 0.0 rpy=-1.5707963 0.0 0.0 -> xyz=0.0 -0.04 0.0 rpy=1.5707963 0.0 0.0
- joint left-thigh-to-knee-ankle-rotor-1: origin xyz=0.0 26.55e-03 0.0 rpy=-1.5707963 0.0 0.0 -> xyz=0.0 26.55e-03 0.0 rpy=1.5707963 0.0 0.0
- joint left-thigh-to-knee-ankle-rotor-2: origin xyz=0.0 -26.55e-03 0.0 rpy=-1.5707963 0.0 -3.1415927 -> xyz=0.0 -26.55e-03 0.0 rpy=-1.5707963 3.1415927 0.0
- joint right-hip-clamp-to-hip-rotor-1: origin xyz=0.0 0.04 0.0 rpy=-1.5707963 0.0 -3.1415927 -> xyz=0.0 0.04 0.0 rpy=-1.5707963 3.1415927 0.0
- joint right-hip-clamp-to-hip-rotor-2: origin xyz=0.0 -0.04 0.0 rpy=-1.5707963 0.0 0.0 -> xyz=0.0 -0.04 0.0 rpy=1.5707963 0.0 0.0
- joint right-thigh-to-knee-ankle-rotor-1: origin xyz=0.0 26.55e-03 0.0 rpy=-1.5707963 0.0 0.0 -> xyz=0.0 26.55e-03 0.0 rpy=1.5707963 0.0 0.0
- joint right-thigh-to-knee-ankle-rotor-2: origin xyz=0.0 -26.55e-03 0.0 rpy=-1.5707963 0.0 -3.1415927 -> xyz=0.0 -26.55e-03 0.0 rpy=-1.5707963 3.1415927 0.0

File: robot-models/tello_legs.xacro (robot description, xacro)
@@ -2,9 +2,10 @@
 <robot name="tello_legs" xmlns:xacro="http://ros.org/wiki/xacro">
     <xacro:include filename="tello_properties.xacro"/>
-    <link name="ground"/>
+    <xacro:property name="base" value="ground"/>
+    <link name="${base}"/>
     <!-- Left Hip Cluster -->
-    <xacro:L_independent_hip_clamp_rotor_joint parent="ground"/>
+    <xacro:L_independent_hip_clamp_rotor_joint parent="${base}"/>
     <xacro:hip_clamp_rotor prefix="left-"/>
-    <xacro:L_dependent_hip_clamp_joint parent="ground"/>
+    <xacro:L_dependent_hip_clamp_joint parent="${base}"/>
     <xacro:hip_clamp prefix="left-"/>
     <!-- Left Hip Differentials -->
@@ -27,7 +28,7 @@
     <xacro:foot prefix="left-"/>
     <!-- Right Hip Cluster -->
-    <xacro:R_independent_hip_clamp_rotor_joint parent="ground"/>
+    <xacro:R_independent_hip_clamp_rotor_joint parent="${base}"/>
     <xacro:hip_clamp_rotor prefix="right-"/>
-    <xacro:R_dependent_hip_clamp_joint parent="ground"/>
+    <xacro:R_dependent_hip_clamp_joint parent="${base}"/>
     <xacro:hip_clamp prefix="right-"/>
     <!-- Right Hip Differentials -->
