Commit message: Fixes to tello:
- fix joint rpy
- change arm sequence to left,right for consistency
- add separate left,right arm link inertia
- add separate left,right arm link origin

File: robot-models/tello_properties.xacro (robot description, xacro)
@@ -5,7 +5,7 @@
     <xacro:property name="Z_AXIS" value="0 0 1"/>
     <xacro:property name="RPY_up" value="0.0 0.0 0.0"/>
-    <xacro:property name="RPY_down" value="-3.1415927 0.0 0.0"/>
-    <xacro:property name="RPY_left" value="-1.5707963 0.0 -3.1415927"/>
-    <xacro:property name="RPY_right" value="-1.5707963 0.0 0.0"/>
+    <xacro:property name="RPY_down" value="3.1415927 0.0 0.0"/>
+    <xacro:property name="RPY_left" value="-1.5707963 3.1415927 0.0"/>
+    <xacro:property name="RPY_right" value="1.5707963 0.0 0.0"/>
     <xacro:property name="effort_limit" value="150"/>
     <xacro:property name="velocity_limit" value="100"/>
@@ -99,37 +99,53 @@
     <xacro:property name="shoulder_ry_mass" value="0.788506"/>
     <xacro:property name="shoulder_ry_axis" value="${Y_AXIS}"/>
-    <xacro:property name="L_shoulder_ry_joint_xyz" value="0.01346 -0.17608 0.24657"/>
-    <xacro:property name="R_shoulder_ry_joint_xyz" value="0.01346 0.17608 0.24657"/>
+    <xacro:property name="R_shoulder_ry_joint_xyz" value="0.01346 -0.17608 0.24657"/>
+    <xacro:property name="L_shoulder_ry_joint_xyz" value="0.01346 0.17608 0.24657"/>
     <xacro:property name="shoulder_ry_joint_rpy" value="${RPY_up}"/>
-    <xacro:property name="shoulder_ry_origin_xyz" value="0.009265, 0.052623, -0.0001249"/>
-    <xacro:macro name="shoulder_ry_inertia">
+    <xacro:property name="L_shoulder_ry_origin_xyz" value="0.009265 0.052623 -0.0001249"/>
+    <xacro:property name="R_shoulder_ry_origin_xyz" value="0.009265 -0.052623 -0.0001249"/>
+    <xacro:macro name="L_shoulder_ry_inertia">
         <inertia ixx="0.0013678" ixy="0.0000266" ixz="0.0000021" iyy="0.0007392" iyz="-0.0000012" izz="0.000884"/>
+    </xacro:macro>
+    <xacro:macro name="R_shoulder_ry_inertia">
+        <inertia ixx="0.0013678" ixy="-0.0000266" ixz="0.0000021" iyy="0.0007392" iyz="0.0000012" izz="0.000884"/>
     </xacro:macro>
     <xacro:property name="shoulder_rx_mass" value="0.80125"/>
     <xacro:property name="shoulder_rx_axis" value="${X_AXIS}"/>
-    <xacro:property name="L_shoulder_rx_joint_xyz" value="0.0 -0.0575 0.0"/>
-    <xacro:property name="R_shoulder_rx_joint_xyz" value="0.0 0.0575 0.0"/>
+    <xacro:property name="R_shoulder_rx_joint_xyz" value="0.0 -0.0575 0.0"/>
+    <xacro:property name="L_shoulder_rx_joint_xyz" value="0.0 0.0575 0.0"/>
     <xacro:property name="shoulder_rx_joint_rpy" value="${RPY_up}"/>
-    <xacro:property name="shoulder_rx_origin_xyz" value="0.0006041 0.0001221 -0.082361"/>
-    <xacro:macro name="shoulder_rx_inertia">
+    <xacro:property name="L_shoulder_rx_origin_xyz" value="0.0006041 0.0001221 -0.082361"/>
+    <xacro:property name="R_shoulder_rx_origin_xyz" value="0.0006041 -0.0001221 -0.082361"/>
+    <xacro:macro name="L_shoulder_rx_inertia">
         <inertia ixx="0.0011524" ixy="0.0000007" ixz="0.0000396" iyy="0.0011921" iyz="0.0000014" izz="0.0012386"/>
+    </xacro:macro>
+    <xacro:macro name="R_shoulder_rx_inertia">
+        <inertia ixx="0.0011524" ixy="-0.0000007" ixz="0.0000396" iyy="0.0011921" iyz="-0.0000014" izz="0.0012386"/>
     </xacro:macro>
     <xacro:property name="shoulder_rz_mass" value="0.905588"/>
     <xacro:property name="shoulder_rz_axis" value="${Z_AXIS}"/>
+    <xacro:property name="R_shoulder_rz_joint_xyz" value="0.0 0.0 -0.1025"/>
     <xacro:property name="L_shoulder_rz_joint_xyz" value="0.0 0.0 -0.1025"/>
-    <xacro:property name="R_shoulder_rz_joint_xyz" value="0.0 0.0 -0.1025"/>
     <xacro:property name="shoulder_rz_joint_rpy" value="${RPY_up}"/>
-    <xacro:property name="shoulder_rz_origin_xyz" value="0.0001703 -0.016797 -0.060"/>
-    <xacro:macro name="shoulder_rz_inertia">
+    <xacro:property name="L_shoulder_rz_origin_xyz" value="0.0001703 -0.016797 -0.060"/>
+    <xacro:property name="R_shoulder_rz_origin_xyz" value="0.0001703 0.016797 -0.060"/>
+    <xacro:macro name="L_shoulder_rz_inertia">
         <inertia ixx="0.0012713" ixy="0.000001" ixz="-0.000008" iyy="0.0017477" iyz="-0.0000225" izz="0.0008191"/>
+    </xacro:macro>
+    <xacro:macro name="R_shoulder_rz_inertia">
+        <inertia ixx="0.0012713" ixy="-0.000001" ixz="-0.000008" iyy="0.0017477" iyz="0.0000225" izz="0.0008191"/>
     </xacro:macro>
     <xacro:property name="elbow_mass" value="0.34839"/>
     <xacro:property name="elbow_axis" value="${Y_AXIS}"/>
+    <xacro:property name="R_elbow_joint_xyz" value="0.0 0.0 -0.1455"/>
     <xacro:property name="L_elbow_joint_xyz" value="0.0 0.0 -0.1455"/>
-    <xacro:property name="R_elbow_joint_xyz" value="0.0 0.0 -0.1455"/>
     <xacro:property name="elbow_joint_rpy" value="${RPY_up}"/>
-    <xacro:property name="elbow_origin_xyz" value="-0.0059578 0.000111 -0.0426735"/>
-    <xacro:macro name="elbow_inertia">
+    <xacro:property name="L_elbow_origin_xyz" value="-0.0059578 0.000111 -0.0426735"/>
+    <xacro:property name="R_elbow_origin_xyz" value="-0.0059578 -0.000111 -0.0426735"/>
+    <xacro:macro name="L_elbow_inertia">
         <inertia ixx="0.001570" ixy="0.0000002" ixz="0.0000335" iyy="0.0016167" iyz="0.000003" izz="0.0000619"/>
+    </xacro:macro>
+    <xacro:macro name="R_elbow_inertia">
+        <inertia ixx="0.001570" ixy="-0.0000002" ixz="0.0000335" iyy="0.0016167" iyz="-0.000003" izz="0.0000619"/>
     </xacro:macro>
     <xacro:property name="arm_rotor_mass" value="0.0"/>
@@ -146,24 +162,24 @@
     <xacro:property name="shoulder_ry_rotor_mass" value="${arm_rotor_mass}"/>
     <xacro:property name="shoulder_ry_rotor_axis" value="${Y_AXIS}"/>
-    <xacro:property name="L_shoulder_ry_rotor_joint_xyz" value="0.01346 -0.16 0.24657"/>
-    <xacro:property name="R_shoulder_ry_rotor_joint_xyz" value="0.01346 0.16 0.24657"/>
+    <xacro:property name="R_shoulder_ry_rotor_joint_xyz" value="0.01346 -0.16 0.24657"/>
+    <xacro:property name="L_shoulder_ry_rotor_joint_xyz" value="0.01346 0.16 0.24657"/>
     <xacro:property name="shoulder_ry_rotor_joint_rpy" value="${RPY_up}"/>
     <xacro:property name="shoulder_ry_rotor_origin_xyz" value="${arm_rotor_origin}"/>
     <xacro:property name="shoulder_rx_rotor_mass" value="${arm_rotor_mass}"/>
     <xacro:property name="shoulder_rx_rotor_axis" value="${X_AXIS}"/>
-    <xacro:property name="L_shoulder_rx_rotor_joint_xyz" value="0.0 -0.0575 0.0"/>
-    <xacro:property name="R_shoulder_rx_rotor_joint_xyz" value="0.0 0.0575 0.0"/>
+    <xacro:property name="R_shoulder_rx_rotor_joint_xyz" value="0.0 -0.0575 0.0"/>
+    <xacro:property name="L_shoulder_rx_rotor_joint_xyz" value="0.0 0.0575 0.0"/>
     <xacro:property name="shoulder_rx_rotor_joint_rpy" value="${RPY_up}"/>
     <xacro:property name="shoulder_rx_rotor_origin_xyz" value="${arm_rotor_origin}"/>
     <xacro:property name="shoulder_rz_rotor_mass" value="${arm_rotor_mass}"/>
     <xacro:property name="shoulder_rz_rotor_axis" value="${Z_AXIS}"/>
+    <xacro:property name="R_shoulder_rz_rotor_joint_xyz" value="0.0 0.0 -0.1025"/>
     <xacro:property name="L_shoulder_rz_rotor_joint_xyz" value="0.0 0.0 -0.1025"/>
-    <xacro:property name="R_shoulder_rz_rotor_joint_xyz" value="0.0 0.0 -0.1025"/>
     <xacro:property name="shoulder_rz_rotor_joint_rpy" value="${RPY_up}"/>
     <xacro:property name="shoulder_rz_rotor_origin_xyz" value="${arm_rotor_origin}"/>
     <xacro:property name="elbow_rotor_mass" value="${arm_rotor_mass}"/>
     <xacro:property name="elbow_rotor_axis" value="${Y_AXIS}"/>
-    <xacro:property name="L_elbow_rotor_joint_xyz" value="0.0 0.0325 -0.06"/>
-    <xacro:property name="R_elbow_rotor_joint_xyz" value="0.0 -0.0325 -0.06"/>
+    <xacro:property name="R_elbow_rotor_joint_xyz" value="0.0 0.0325 -0.06"/>
+    <xacro:property name="L_elbow_rotor_joint_xyz" value="0.0 -0.0325 -0.06"/>
     <xacro:property name="elbow_rotor_joint_rpy" value="${RPY_up}"/>
     <xacro:property name="elbow_rotor_origin_xyz" value="${arm_rotor_origin}"/>
@@ -602,10 +618,19 @@
                                origin_rpy="${shoulder_ry_joint_rpy}"/>
     </xacro:macro>
-    <xacro:macro name="shoulder_ry" params="prefix">
-        <link name="${prefix}shoulder-ry">
+    <xacro:macro name="left_shoulder_ry">
+        <link name="left-shoulder-ry">
             <inertial>
                 <mass value="${shoulder_ry_mass}"/>
-                <origin xyz="${shoulder_ry_origin_xyz}"/>
-                <xacro:shoulder_ry_inertia/>
+                <origin xyz="${L_shoulder_ry_origin_xyz}"/>
+                <xacro:L_shoulder_ry_inertia/>
+            </inertial>
+        </link>
+    </xacro:macro>
+    <xacro:macro name="right_shoulder_ry">
+        <link name="right-shoulder-ry">
+            <inertial>
+                <mass value="${shoulder_ry_mass}"/>
+                <origin xyz="${R_shoulder_ry_origin_xyz}"/>
+                <xacro:R_shoulder_ry_inertia/>
             </inertial>
         </link>
@@ -649,5 +674,5 @@
     </xacro:macro>
     <xacro:macro name="L_independent_shoulder_rx_joint" params="parent">
-        <xacro:independent_joint name="${parent}-to-left-shoulder-rx"
+        <xacro:independent_joint name="${parent}-to-shoulder-rx"
                                parent="${parent}" child="left-shoulder-rx"
                                axis="${shoulder_rx_axis}"
@@ -656,5 +681,5 @@
     </xacro:macro>
     <xacro:macro name="L_dependent_shoulder_rx_joint" params="parent">
-        <xacro:dependent_joint name="${parent}-to-left-shoulder-rx"
+        <xacro:dependent_joint name="${parent}-to-shoulder-rx"
                                parent="${parent}" child="left-shoulder-rx"
                                axis="${shoulder_rx_axis}"
@@ -663,5 +688,5 @@
     </xacro:macro>
    <xacro:macro name="R_independent_shoulder_rx_joint" params="parent">
-        <xacro:independent_joint name="${parent}-to-right-shoulder-rx"
+        <xacro:independent_joint name="${parent}-to-shoulder-rx"
                                parent="${parent}" child="right-shoulder-rx"
                                axis="${shoulder_rx_axis}"
@@ -670,5 +695,5 @@
     </xacro:macro>
     <xacro:macro name="R_dependent_shoulder_rx_joint" params="parent">
-        <xacro:dependent_joint name="${parent}-to-right-shoulder-rx"
+        <xacro:dependent_joint name="${parent}-to-shoulder-rx"
                                parent="${parent}" child="right-shoulder-rx"
                                axis="${shoulder_rx_axis}"
@@ -676,15 +701,24 @@
                                origin_rpy="${shoulder_rx_joint_rpy}"/>
     </xacro:macro>
-    <xacro:macro name="shoulder_rx" params="prefix">
-        <link name="${prefix}shoulder-rx">
+    <xacro:macro name="left_shoulder_rx">
+        <link name="left-shoulder-rx">
             <inertial>
                 <mass value="${shoulder_rx_mass}"/>
-                <origin xyz="${shoulder_rx_origin_xyz}"/>
-                <xacro:shoulder_rx_inertia/>
+                <origin xyz="${L_shoulder_rx_origin_xyz}"/>
+                <xacro:L_shoulder_rx_inertia/>
+            </inertial>
+        </link>
+    </xacro:macro>
+    <xacro:macro name="right_shoulder_rx">
+        <link name="right-shoulder-rx">
+            <inertial>
+                <mass value="${shoulder_rx_mass}"/>
+                <origin xyz="${R_shoulder_rx_origin_xyz}"/>
+                <xacro:R_shoulder_rx_inertia/>
             </inertial>
         </link>
     </xacro:macro>
     <xacro:macro name="L_independent_shoulder_rx_rotor_joint" params="parent">
-        <xacro:independent_joint name="${parent}-to-left-shoulder-rx-rotor"
+        <xacro:independent_joint name="${parent}-to-shoulder-rx-rotor"
                                parent="${parent}" child="left-shoulder-rx-rotor"
                                axis="${shoulder_rx_rotor_axis}"
@@ -693,5 +727,5 @@
     </xacro:macro>
     <xacro:macro name="L_dependent_shoulder_rx_rotor_joint" params="parent">
-        <xacro:dependent_joint name="${parent}-to-left-shoulder-rx-rotor"
+        <xacro:dependent_joint name="${parent}-to-shoulder-rx-rotor"
                                parent="${parent}" child="left-shoulder-rx-rotor"
                                axis="${shoulder_rx_rotor_axis}"
@@ -700,5 +734,5 @@
     </xacro:macro>
    <xacro:macro name="R_independent_shoulder_rx_rotor_joint" params="parent">
-        <xacro:independent_joint name="${parent}-to-right-shoulder-rx-rotor"
+        <xacro:independent_joint name="${parent}-to-shoulder-rx-rotor"
                                parent="${parent}" child="right-shoulder-rx-rotor"
                                axis="${shoulder_rx_rotor_axis}"
@@ -707,5 +741,5 @@
     </xacro:macro>
     <xacro:macro name="R_dependent_shoulder_rx_rotor_joint" params="parent">
-        <xacro:dependent_joint name="${parent}-to-right-shoulder-rx-rotor"
+        <xacro:dependent_joint name="${parent}-to-shoulder-rx-rotor"
                                parent="${parent}" child="right-shoulder-rx-rotor"
                                axis="${shoulder_rx_rotor_axis}"
@@ -723,5 +757,5 @@
     </xacro:macro>
     <xacro:macro name="L_independent_shoulder_rz_joint" params="parent">
-        <xacro:independent_joint name="${parent}-to-left-shoulder-rz"
+        <xacro:independent_joint name="${parent}-to-shoulder-rz"
                                parent="${parent}" child="left-shoulder-rz"
                                axis="${shoulder_rz_axis}"
@@ -730,5 +764,5 @@
     </xacro:macro>
     <xacro:macro name="L_dependent_shoulder_rz_joint" params="parent">
-        <xacro:dependent_joint name="${parent}-to-left-shoulder-rz"
+        <xacro:dependent_joint name="${parent}-to-shoulder-rz"
                                parent="${parent}" child="left-shoulder-rz"
                                axis="${shoulder_rz_axis}"
@@ -737,5 +771,5 @@
     </xacro:macro>
    <xacro:macro name="R_independent_shoulder_rz_joint" params="parent">
-        <xacro:independent_joint name="${parent}-to-right-shoulder-rz"
+        <xacro:independent_joint name="${parent}-to-shoulder-rz"
                                parent="${parent}" child="right-shoulder-rz"
                                axis="${shoulder_rz_axis}"
@@ -744,5 +778,5 @@
     </xacro:macro>
     <xacro:macro name="R_dependent_shoulder_rz_joint" params="parent">
-        <xacro:dependent_joint name="${parent}-to-right-shoulder-rz"
+        <xacro:dependent_joint name="${parent}-to-shoulder-rz"
                                parent="${parent}" child="right-shoulder-rz"
                                axis="${shoulder_rz_axis}"
@@ -750,15 +784,24 @@
                                origin_rpy="${shoulder_rz_joint_rpy}"/>
     </xacro:macro>
-    <xacro:macro name="shoulder_rz" params="prefix">
-        <link name="${prefix}shoulder-rz">
+    <xacro:macro name="left_shoulder_rz">
+        <link name="left-shoulder-rz">
             <inertial>
                 <mass value="${shoulder_rz_mass}"/>
-                <origin xyz="${shoulder_rz_origin_xyz}"/>
-                <xacro:shoulder_rz_inertia/>
+                <origin xyz="${L_shoulder_rz_origin_xyz}"/>
+                <xacro:L_shoulder_rz_inertia/>
+            </inertial>
+        </link>
+    </xacro:macro>
+    <xacro:macro name="right_shoulder_rz">
+        <link name="right-shoulder-rz">
+            <inertial>
+                <mass value="${shoulder_rz_mass}"/>
+                <origin xyz="${R_shoulder_rz_origin_xyz}"/>
+                <xacro:R_shoulder_rz_inertia/>
             </inertial>
         </link>
     </xacro:macro>
     <xacro:macro name="L_independent_shoulder_rz_rotor_joint" params="parent">
-        <xacro:independent_joint name="${parent}-to-left-shoulder-rz-rotor"
+        <xacro:independent_joint name="${parent}-to-shoulder-rz-rotor"
                                parent="${parent}" child="left-shoulder-rz-rotor"
                                axis="${shoulder_rz_rotor_axis}"
@@ -767,5 +810,5 @@
     </xacro:macro>
     <xacro:macro name="L_dependent_shoulder_rz_rotor_joint" params="parent">
-        <xacro:dependent_joint name="${parent}-to-left-shoulder-rz-rotor"
+        <xacro:dependent_joint name="${parent}-to-shoulder-rz-rotor"
                                parent="${parent}" child="left-shoulder-rz-rotor"
                                axis="${shoulder_rz_rotor_axis}"
@@ -774,5 +817,5 @@
     </xacro:macro>
    <xacro:macro name="R_independent_shoulder_rz_rotor_joint" params="parent">
-        <xacro:independent_joint name="${parent}-to-right-shoulder-rz-rotor"
+        <xacro:independent_joint name="${parent}-to-shoulder-rz-rotor"
                                parent="${parent}" child="right-shoulder-rz-rotor"
                                axis="${shoulder_rz_rotor_axis}"
@@ -781,5 +824,5 @@
     </xacro:macro>
     <xacro:macro name="R_dependent_shoulder_rz_rotor_joint" params="parent">
-        <xacro:dependent_joint name="${parent}-to-right-shoulder-rz-rotor"
+        <xacro:dependent_joint name="${parent}-to-shoulder-rz-rotor"
                                parent="${parent}" child="right-shoulder-rz-rotor"
                                axis="${shoulder_rz_rotor_axis}"
@@ -797,5 +840,5 @@
     </xacro:macro>
     <xacro:macro name="L_independent_elbow_joint" params="parent">
-        <xacro:independent_joint name="${parent}-to-left-elbow"
+        <xacro:independent_joint name="${parent}-to-elbow"
                                parent="${parent}" child="left-elbow"
                                axis="${elbow_axis}"
@@ -804,5 +847,5 @@
     </xacro:macro>
     <xacro:macro name="L_dependent_elbow_joint" params="parent">
-        <xacro:dependent_joint name="${parent}-to-left-elbow"
+        <xacro:dependent_joint name="${parent}-to-elbow"
                                parent="${parent}" child="left-elbow"
                                axis="${elbow_axis}"
@@ -811,5 +854,5 @@
     </xacro:macro>
    <xacro:macro name="R_independent_elbow_joint" params="parent">
-        <xacro:independent_joint name="${parent}-to-right-elbow"
+        <xacro:independent_joint name="${parent}-to-elbow"
                                parent="${parent}" child="right-elbow"
                                axis="${elbow_axis}"
@@ -818,5 +861,5 @@
     </xacro:macro>
     <xacro:macro name="R_dependent_elbow_joint" params="parent">
-        <xacro:dependent_joint name="${parent}-to-right-elbow"
+        <xacro:dependent_joint name="${parent}-to-elbow"
                                parent="${parent}" child="right-elbow"
                                axis="${elbow_axis}"
@@ -824,15 +867,24 @@
                                origin_rpy="${elbow_joint_rpy}"/>
     </xacro:macro>
-    <xacro:macro name="elbow" params="prefix">
-        <link name="${prefix}elbow">
+    <xacro:macro name="left_elbow">
+        <link name="left-elbow">
             <inertial>
                 <mass value="${elbow_mass}"/>
-                <origin xyz="${elbow_origin_xyz}"/>
-                <xacro:elbow_inertia/>
+                <origin xyz="${L_elbow_origin_xyz}"/>
+                <xacro:L_elbow_inertia/>
+            </inertial>
+        </link>
+    </xacro:macro>
+    <xacro:macro name="right_elbow">
+        <link name="right-elbow">
+            <inertial>
+                <mass value="${elbow_mass}"/>
+                <origin xyz="${R_elbow_origin_xyz}"/>
+                <xacro:R_elbow_inertia/>
             </inertial>
         </link>
     </xacro:macro>
     <xacro:macro name="L_independent_elbow_rotor_joint" params="parent">
-        <xacro:independent_joint name="${parent}-to-left-elbow-rotor"
+        <xacro:independent_joint name="${parent}-to-elbow-rotor"
                                parent="${parent}" child="left-elbow-rotor"
                                axis="${elbow_rotor_axis}"
@@ -841,5 +893,5 @@
     </xacro:macro>
     <xacro:macro name="L_dependent_elbow_rotor_joint" params="parent">
-        <xacro:dependent_joint name="${parent}-to-left-elbow-rotor"
+        <xacro:dependent_joint name="${parent}-to-elbow-rotor"
                                parent="${parent}" child="left-elbow-rotor"
                                axis="${elbow_rotor_axis}"
@@ -848,5 +900,5 @@
     </xacro:macro>
    <xacro:macro name="R_independent_elbow_rotor_joint" params="parent">
-        <xacro:independent_joint name="${parent}-to-right-elbow-rotor"
+        <xacro:independent_joint name="${parent}-to-elbow-rotor"
                                parent="${parent}" child="right-elbow-rotor"
                                axis="${elbow_rotor_axis}"
@@ -855,5 +907,5 @@
     </xacro:macro>
     <xacro:macro name="R_dependent_elbow_rotor_joint" params="parent">
-        <xacro:dependent_joint name="${parent}-to-right-elbow-rotor"
+        <xacro:dependent_joint name="${parent}-to-elbow-rotor"
                                parent="${parent}" child="right-elbow-rotor"
                                axis="${elbow_rotor_axis}"
