Commit message: Upgrade minimum cmake version in googletest folder

File: robot-models/mit_humanoid_leg.xacro (robot description, xacro)
@@ -169,4 +169,20 @@
     <!-- Ankle Flexion/Extension -->
     <xacro:macro name="ankle" params="prefix y_sign">
+        <joint name="${prefix}hipy_to_ankle_rotor" type="revolute" independent="false">
+            <axis xyz="0 1 0"/>
+            <origin xyz=".01563 ${y_sign * -.0454} -.13354"/>
+            <parent link="${prefix}hip_ry_link"/>
+            <child link="${prefix}ankle_rotor"/>
+            <limit effort="${effort_limit}" velocity="${velocity_limit}"
+                   lower="${joint_lower_limit}" upper="${joint_upper_limit}"/>
+        </joint>
+        <link name="${prefix}ankle_rotor">
+            <inertial>
+                <mass value="0."/>
+                <origin xyz="0. 0. 0."/>
+                <inertia ixx="1.084e-4" ixy="0.0" ixz="0.0"
+                         iyy="1.6841e-4" iyz="0.0" izz="1.084e-4"/>
+            </inertial>
+        </link>
         <joint name="${prefix}knee_to_ankle" type="revolute">
             <axis xyz="0 1 0"/>
@@ -183,20 +199,4 @@
                 <inertia ixx="0.0000842" ixy="0.0" ixz="-0.0000488"
                          iyy="0.0007959" iyz="0.0" izz="0.0007681"/>
-            </inertial>
-        </link>
-        <joint name="${prefix}hipy_to_ankle_rotor" type="revolute" independent="false">
-            <axis xyz="0 1 0"/>
-            <origin xyz=".01563 ${y_sign * -.0454} -.13354"/>
-            <parent link="${prefix}hip_ry_link"/>
-            <child link="${prefix}ankle_rotor"/>
-            <limit effort="${effort_limit}" velocity="${velocity_limit}"
-                   lower="${joint_lower_limit}" upper="${joint_upper_limit}"/>
-        </joint>
-        <link name="${prefix}ankle_rotor">
-            <inertial>
-                <mass value="0."/>
-                <origin xyz="0. 0. 0."/>
-                <inertia ixx="1.084e-4" ixy="0.0" ixz="0.0"
-                         iyy="1.6841e-4" iyz="0.0" izz="1.084e-4"/>
             </inertial>
         </link>
