Commit message: Update urdfs

File: robot-models/mit_humanoid.urdf (robot description, URDF)
Before this commit: robot mit_humanoid, 37 links, 36 joints
Links:
- link left_knee_link: mass 0.35434 -> 0.35435
- link right_knee_link: mass 0.35434 -> 0.35435

File: robot-models/mit_humanoid_leg.urdf (robot description, URDF)
Before this commit: robot mit_humanoid_leg, 11 links, 10 joints
Links:
- link knee_link: mass 0.35434 -> 0.35435

Commit message: Corrected rotor mass for humanoid

File: robot-models/mit_humanoid.urdf (robot description, URDF)
Before this commit: robot mit_humanoid, 37 links, 36 joints
Links:
- link left_ankle_rotor: mass 0.001 -> 0.05
- link left_elbow_rotor: mass 0.001 -> 0.05
- link left_hip_rx_rotor: mass 0.001 -> 0.05
- link left_hip_ry_rotor: mass 0.0025 -> 0.1
- link left_hip_rz_rotor: mass 0.001 -> 0.05
- link left_knee_rotor: mass 0.0025 -> 0.1
- link left_shoulder_rx_rotor: mass 0.001 -> 0.05
- link left_shoulder_ry_rotor: mass 0.001 -> 0.05
- link left_shoulder_rz_rotor: mass 0.001 -> 0.05
- link right_ankle_rotor: mass 0.001 -> 0.05
- link right_elbow_rotor: mass 0.001 -> 0.05
- link right_hip_rx_rotor: mass 0.001 -> 0.05
- link right_hip_ry_rotor: mass 0.0025 -> 0.1
- link right_hip_rz_rotor: mass 0.001 -> 0.05
- link right_knee_rotor: mass 0.0025 -> 0.1
- link right_shoulder_rx_rotor: mass 0.001 -> 0.05
- link right_shoulder_ry_rotor: mass 0.001 -> 0.05
- link right_shoulder_rz_rotor: mass 0.001 -> 0.05

File: robot-models/mit_humanoid.xacro (robot description, xacro)
@@ -26,5 +26,5 @@
         <link name="${prefix}hip_rz_rotor">
             <inertial>
-                <mass value="0.001"/>
+                <mass value="0.05"/>
                 <origin xyz="0. 0. 0."/>
                 <inertia ixx="1.084e-4" ixy="0.0" ixz="0.0"
@@ -63,5 +63,5 @@
         <link name="${prefix}hip_rx_rotor">
             <inertial>
-                <mass value="0.001"/>
+                <mass value="0.05"/>
                 <origin xyz="0. 0. 0."/>
                 <inertia ixx="1.6841e-4" ixy="0.0" ixz="0.0"
@@ -99,5 +99,5 @@
         <link name="${prefix}hip_ry_rotor">
             <inertial>
-                <mass value="0.0025"/>
+                <mass value="0.1"/>
                 <origin xyz="0. 0. 0."/>
                 <inertia ixx="3.443e-4" ixy="0.0" ixz="0.0"
@@ -135,5 +135,5 @@
         <link name="${prefix}knee_rotor">
             <inertial>
-                <mass value="0.0025"/>
+                <mass value="0.1"/>
                 <origin xyz="0. 0. 0."/>
                 <inertia ixx="3.443e-4" ixy="0.0" ixz="0.0"
@@ -157,5 +157,5 @@
         <link name="${prefix}ankle_rotor">
             <inertial>
-                <mass value="0.001"/>
+                <mass value="0.05"/>
                 <origin xyz="0. 0. 0."/>
                 <inertia ixx="1.084e-4" ixy="0.0" ixz="0.0"
@@ -207,5 +207,5 @@
         <link name="${prefix}shoulder_ry_rotor">
             <inertial>
-                <mass value="0.001"/>
+                <mass value="0.05"/>
                 <origin xyz="0. 0. 0."/>
                 <inertia ixx="1.084e-4" ixy="0.0" ixz="0.0"
@@ -243,5 +243,5 @@
         <link name="${prefix}shoulder_rx_rotor">
             <inertial>
-                <mass value="0.001"/>
+                <mass value="0.05"/>
                 <origin xyz="0. 0. 0."/>
                 <inertia ixx="1.6841e-4" ixy="0.0" ixz="0.0"
@@ -279,5 +279,5 @@
         <link name="${prefix}shoulder_rz_rotor">
             <inertial>
-                <mass value="0.001"/>
+                <mass value="0.05"/>
                 <origin xyz="0. 0. 0."/>
                 <inertia ixx="1.084e-4" ixy="0.0" ixz="0.0"
@@ -315,5 +315,5 @@
         <link name="${prefix}elbow_rotor">
             <inertial>
-                <mass value="0.001"/>
+                <mass value="0.05"/>
                 <origin xyz="0. 0. 0."/>
                 <inertia ixx="1.084e-4" ixy="0.0" ixz="0.0"

Commit message: Fix ankle rotor position

File: robot-models/mit_humanoid.urdf (robot description, URDF)
Before this commit: robot mit_humanoid, 37 links, 36 joints
Joints:
- joint left_hipy_to_ankle_rotor: origin xyz=0. 0. 0. -> xyz=.01563 0.0454 -.13354
- joint right_hipy_to_ankle_rotor: origin xyz=0. 0. 0. -> xyz=.01563 -0.0454 -.13354

File: robot-models/mit_humanoid.xacro (robot description, xacro)
@@ -151,5 +151,5 @@
         <joint name="${prefix}hipy_to_ankle_rotor" type="continuous" independent="false">
             <axis xyz="0 1 0"/>
-            <origin xyz="0. 0. 0."/>
+            <origin xyz=".01563 ${y_sign * -.0454} -.13354"/>
             <parent link="${prefix}hip_ry_link"/>
             <child link="${prefix}ankle_rotor"/>

File: robot-models/mit_humanoid_leg.urdf (robot description, URDF)
Before this commit: robot mit_humanoid_leg, 11 links, 10 joints
Joints:
- joint hipy_to_ankle_rotor: origin xyz=0. 0. 0. -> xyz=.01563 -0.0454 -.13354

File: robot-models/mit_humanoid_leg.xacro (robot description, xacro)
@@ -151,5 +151,5 @@
         <joint name="${prefix}hipy_to_ankle_rotor" type="continuous" independent="false">
             <axis xyz="0 1 0"/>
-            <origin xyz="0. 0. 0."/>
+            <origin xyz=".01563 ${y_sign * -.0454} -.13354"/>
             <parent link="${prefix}hip_ry_link"/>
             <child link="${prefix}ankle_rotor"/>

Commit message: WIP

File: robot-models/mit_humanoid.urdf (robot description, URDF)
Before this commit: robot mit_humanoid, 37 links, 36 joints
Links:
- added link ground
Joints:
- added joint world_to_base: type floating, parent ground, child Floating Base, origin xyz=0 0 0 rpy=0 0 0

File: robot-models/mit_humanoid.xacro (robot description, xacro)
@@ -368,4 +368,5 @@
     </xacro:macro>
     <!-- End of macro definitions -->
+    <link name="ground"/>
     <link name="Floating Base">
         <inertial>
@@ -376,4 +377,9 @@
         </inertial>
     </link>
+    <joint name="world_to_base" type="floating">
+        <origin xyz="0 0 0" rpy="0 0 0"/>
+        <parent link="ground"/>
+        <child link="Floating Base"/>
+    </joint>
     <xacro:hipz prefix="right_" y_sign="1"/>
     <xacro:hipz prefix="left_" y_sign="-1"/>
