Commit message: Benchmarks work with new urdf floating base compatibility

File: robot-models/jvrc1_humanoid.urdf (robot description, URDF)
Before this commit: robot jvrc1_humanoid, 58 links, 57 joints
Links:
- added link pelvis, mass 10
- link base: mass 10 -> None
Joints:
- removed joint base-to-left-hip-pitch
- removed joint base-to-left-hip-pitch-rotor
- removed joint base-to-right-hip-pitch
- removed joint base-to-right-hip-pitch-rotor
- removed joint base-to-waist-yaw
- removed joint base-to-waist-yaw-rotor
- added joint base_to_pelvis: type floating, parent base, child pelvis, origin xyz=0 0 0 rpy=0 0 0
- added joint pelvis-to-left-hip-pitch: type revolute, parent pelvis, child left-hip-pitch, origin xyz=0.0 0.096 0.0 rpy=0.0 0.0 0.0, axis 0 1 0, limit lower=-10 upper=10 effort=150 velocity=100
- added joint pelvis-to-left-hip-pitch-rotor: type revolute, parent pelvis, child left-hip-pitch-rotor, origin xyz=0.0 0.096 0.0 rpy=0.0 0.0 0.0, axis 0 1 0, limit lower=-10 upper=10 effort=150 velocity=100
- added joint pelvis-to-right-hip-pitch: type revolute, parent pelvis, child right-hip-pitch, origin xyz=0.0 -0.096 -87e-03 rpy=0.0 0.0 0.0, axis 0 1 0, limit lower=-10 upper=10 effort=150 velocity=100
- added joint pelvis-to-right-hip-pitch-rotor: type revolute, parent pelvis, child right-hip-pitch-rotor, origin xyz=0.0 -0.096 -87e-03 rpy=0.0 0.0 0.0, axis 0 1 0, limit lower=-10 upper=10 effort=150 velocity=100
- added joint pelvis-to-waist-yaw: type revolute, parent pelvis, child waist-yaw, origin xyz=0.0 0.0 0.192 rpy=0.0 0.0 0.0, axis 0 0 1, limit lower=-10 upper=10 effort=150 velocity=100
- added joint pelvis-to-waist-yaw-rotor: type revolute, parent pelvis, child waist-yaw-rotor, origin xyz=0.0 0.0 0.192 rpy=0.0 0.0 0.0, axis 0 0 1, limit lower=-10 upper=10 effort=150 velocity=100

File: robot-models/jvrc1_humanoid.xacro (robot description, xacro)
@@ -3,8 +3,14 @@
     <xacro:include filename="jvrc1_properties.xacro"/>
     <xacro:property name="base" value="base"/>
-    <xacro:pelvis name="${base}"/>
-    <xacro:independent_waist_yaw_joint parent="${base}"/>
+    <link name="${base}"/>
+    <xacro:pelvis name="pelvis"/>
+    <joint name="base_to_pelvis" type="floating">
+        <origin xyz="0 0 0" rpy="0 0 0"/>
+        <parent link="${base}"/>
+        <child link="pelvis"/>
+    </joint>
+    <xacro:independent_waist_yaw_joint parent="pelvis"/>
     <xacro:waist_yaw/>
-    <xacro:dependent_waist_yaw_rotor_joint parent="${base}"/>
+    <xacro:dependent_waist_yaw_rotor_joint parent="pelvis"/>
     <xacro:waist_yaw_rotor/>
     <xacro:trans_constraint name="waist-yaw-transmission"
@@ -47,7 +53,7 @@
                             successor="neck-pitch-rotor"/> -->
     <!-- Left Leg -->
-    <xacro:L_independent_hip_pitch_joint parent="${base}"/>
+    <xacro:L_independent_hip_pitch_joint parent="pelvis"/>
     <xacro:hip_pitch prefix="left-"/>
-    <xacro:L_dependent_hip_pitch_rotor_joint parent="${base}"/>
+    <xacro:L_dependent_hip_pitch_rotor_joint parent="pelvis"/>
     <xacro:hip_pitch_rotor prefix="left-"/>
     <xacro:trans_constraint name="left-hip-pitch-transmission"
@@ -90,7 +96,7 @@
                             successor="left-ankle-pitch-rotor"/>
     <!-- Right Leg -->
-    <xacro:R_independent_hip_pitch_joint parent="${base}"/>
+    <xacro:R_independent_hip_pitch_joint parent="pelvis"/>
     <xacro:hip_pitch prefix="right-"/>
-    <xacro:R_dependent_hip_pitch_rotor_joint parent="${base}"/>
+    <xacro:R_dependent_hip_pitch_rotor_joint parent="pelvis"/>
     <xacro:hip_pitch_rotor prefix="right-"/>
     <xacro:trans_constraint name="right-hip-pitch-transmission"

File: robot-models/jvrc1_humanoid_approximate.urdf (robot description, URDF)
Before this commit: robot jvrc1_humanoid, 33 links, 32 joints
Links:
- added link pelvis, mass 10
- link base: mass 10 -> None
Joints:
- added joint base_to_pelvis: type floating, parent base, child pelvis, origin xyz=0 0 0 rpy=0 0 0

File: robot-models/jvrc1_humanoid_approximate.xacro (robot description, xacro)
@@ -3,5 +3,11 @@
     <xacro:include filename="jvrc1_properties.xacro"/>
     <xacro:property name="base" value="base"/>
-    <xacro:pelvis name="${base}"/>
+    <link name="${base}"/>
+    <xacro:pelvis name="pelvis"/>
+    <joint name="base_to_pelvis" type="floating">
+        <origin xyz="0 0 0" rpy="0 0 0"/>
+        <parent link="${base}"/>
+        <child link="pelvis"/>
+    </joint>
     <xacro:independent_waist_yaw_joint parent="${base}"/>
     <xacro:waist_yaw/>

File: robot-models/mini_cheetah.urdf (robot description, URDF)
Before this commit: robot mini_cheetah, 25 links, 24 joints
Links:
- added link base
Joints:
- added joint base_to_floating_base: type floating, parent base, child Floating Base, origin xyz=0 0 0 rpy=0 0 0

File: robot-models/mini_cheetah.xacro (robot description, xacro)
@@ -2,4 +2,5 @@
 <robot name="mini_cheetah" xmlns:xacro="http://ros.org/wiki/xacro">
     <xacro:include filename="mini_cheetah_properties.xacro"/>
+    <link name="base"/>
     <link name="Floating Base">
         <inertial>
@@ -11,4 +12,9 @@
         </inertial>
     </link>
+    <joint name="base_to_floating_base" type="floating">
+        <origin xyz="0 0 0" rpy="0 0 0"/>
+        <parent link="base"/>
+        <child link="Floating Base"/>
+    </joint>
     <xacro:abad prefix="FR" x_sign="1" y_sign="-1"/>
     <xacro:hip prefix="FR" x_sign="1" y_sign="-1"/>

File: robot-models/mini_cheetah_approximate.urdf (robot description, URDF)
Before this commit: robot mini_cheetah, 13 links, 12 joints
Links:
- added link base
Joints:
- added joint base_to_floating_base: type floating, parent base, child Floating Base, origin xyz=0 0 0 rpy=0 0 0

File: robot-models/mini_cheetah_approximate.xacro (robot description, xacro)
@@ -2,4 +2,5 @@
 <robot name="mini_cheetah" xmlns:xacro="http://ros.org/wiki/xacro">
     <xacro:include filename="mini_cheetah_properties.xacro"/>
+    <link name="base"/>
     <link name="Floating Base">
         <inertial>
@@ -11,4 +12,9 @@
         </inertial>
     </link>
+    <joint name="base_to_floating_base" type="floating">
+        <origin xyz="0 0 0" rpy="0 0 0"/>
+        <parent link="base"/>
+        <child link="Floating Base"/>
+    </joint>
     <xacro:abad_approx prefix="FR" x_sign="1" y_sign="-1"/>
     <xacro:hip_approx prefix="FR" x_sign="1" y_sign="-1"/>

File: robot-models/mini_cheetah_fl_leg.urdf (robot description, URDF)
Before this commit: robot mini_cheetah_fl_leg, 7 links, 6 joints
Joints:
- joint FL_abad_to_hip_j: limit (none) -> lower=-10 upper=10 effort=150 velocity=100; origin xyz=0 0.062 0.0 rpy=0 0 3.14159265359 -> xyz=0 0.062 0.0 rpy=0 0 3.141592653589793; type continuous -> revolute
- joint FL_abad_to_hip_rotor_j: limit (none) -> lower=-10 upper=10 effort=150 velocity=100; origin xyz=0.0 0.04 0.0 rpy=0 0 3.14159265359 -> xyz=0.0 0.04 0.0 rpy=0 0 3.141592653589793; type continuous -> revolute
- joint FL_hip_to_knee_j: limit (none) -> lower=-10 upper=10 effort=150 velocity=100; type continuous -> revolute
- joint FL_hip_to_knee_rotor_j: limit (none) -> lower=-10 upper=10 effort=150 velocity=100; type continuous -> revolute
- joint torso_to_FL_abad_j: limit (none) -> lower=-10 upper=10 effort=150 velocity=100; type continuous -> revolute
- joint torso_to_FL_abad_rotor_j: limit (none) -> lower=-10 upper=10 effort=150 velocity=100; type continuous -> revolute

File: robot-models/mini_cheetah_fr_leg.urdf (robot description, URDF)
Before this commit: robot mini_cheetah_fr_leg, 7 links, 6 joints
Joints:
- joint FR_abad_to_hip_j: limit (none) -> lower=-10 upper=10 effort=150 velocity=100; origin xyz=0 -0.062 0.0 rpy=0 0 3.14159265359 -> xyz=0 -0.062 0.0 rpy=0 0 3.141592653589793; type continuous -> revolute
- joint FR_abad_to_hip_rotor_j: limit (none) -> lower=-10 upper=10 effort=150 velocity=100; origin xyz=0.0 -0.04 0.0 rpy=0 0 3.14159265359 -> xyz=0.0 -0.04 0.0 rpy=0 0 3.141592653589793; type continuous -> revolute
- joint FR_hip_to_knee_j: limit (none) -> lower=-10 upper=10 effort=150 velocity=100; type continuous -> revolute
- joint FR_hip_to_knee_rotor_j: limit (none) -> lower=-10 upper=10 effort=150 velocity=100; type continuous -> revolute
- joint torso_to_FR_abad_j: limit (none) -> lower=-10 upper=10 effort=150 velocity=100; type continuous -> revolute
- joint torso_to_FR_abad_rotor_j: limit (none) -> lower=-10 upper=10 effort=150 velocity=100; type continuous -> revolute

File: robot-models/mini_cheetah_hl_leg.urdf (robot description, URDF)
Before this commit: robot mini_cheetah_hl_leg, 7 links, 6 joints
Joints:
- joint HL_abad_to_hip_j: limit (none) -> lower=-10 upper=10 effort=150 velocity=100; origin xyz=0 0.062 0.0 rpy=0 0 3.14159265359 -> xyz=0 0.062 0.0 rpy=0 0 3.141592653589793; type continuous -> revolute
- joint HL_abad_to_hip_rotor_j: limit (none) -> lower=-10 upper=10 effort=150 velocity=100; origin xyz=0.0 0.04 0.0 rpy=0 0 3.14159265359 -> xyz=0.0 0.04 0.0 rpy=0 0 3.141592653589793; type continuous -> revolute
- joint HL_hip_to_knee_j: limit (none) -> lower=-10 upper=10 effort=150 velocity=100; type continuous -> revolute
- joint HL_hip_to_knee_rotor_j: limit (none) -> lower=-10 upper=10 effort=150 velocity=100; type continuous -> revolute
- joint torso_to_HL_abad_j: limit (none) -> lower=-10 upper=10 effort=150 velocity=100; type continuous -> revolute
- joint torso_to_HL_abad_rotor_j: limit (none) -> lower=-10 upper=10 effort=150 velocity=100; type continuous -> revolute

File: robot-models/mini_cheetah_hr_leg.urdf (robot description, URDF)
Before this commit: robot mini_cheetah_hr_leg, 7 links, 6 joints
Joints:
- joint HR_abad_to_hip_j: limit (none) -> lower=-10 upper=10 effort=150 velocity=100; origin xyz=0 -0.062 0.0 rpy=0 0 3.14159265359 -> xyz=0 -0.062 0.0 rpy=0 0 3.141592653589793; type continuous -> revolute
- joint HR_abad_to_hip_rotor_j: limit (none) -> lower=-10 upper=10 effort=150 velocity=100; origin xyz=0.0 -0.04 0.0 rpy=0 0 3.14159265359 -> xyz=0.0 -0.04 0.0 rpy=0 0 3.141592653589793; type continuous -> revolute
- joint HR_hip_to_knee_j: limit (none) -> lower=-10 upper=10 effort=150 velocity=100; type continuous -> revolute
- joint HR_hip_to_knee_rotor_j: limit (none) -> lower=-10 upper=10 effort=150 velocity=100; type continuous -> revolute
- joint torso_to_HR_abad_j: limit (none) -> lower=-10 upper=10 effort=150 velocity=100; type continuous -> revolute
- joint torso_to_HR_abad_rotor_j: limit (none) -> lower=-10 upper=10 effort=150 velocity=100; type continuous -> revolute

File: robot-models/mit_humanoid_approximate.urdf (robot description, URDF)
Before this commit: robot mit_humanoid, 19 links, 18 joints
Links:
- added link base
Joints:
- added joint base_to_Floating Base: type floating, parent base, child Floating Base, origin xyz=0 0 0 rpy=0 0 0

File: robot-models/mit_humanoid_approximate.xacro (robot description, xacro)
@@ -179,4 +179,5 @@
     </xacro:macro>
     <!-- End of macro definitions -->
+    <link name="base"/>
     <link name="Floating Base">
         <inertial>
@@ -187,4 +188,9 @@
         </inertial>
     </link>
+    <joint name="base_to_Floating Base" type="floating">
+        <origin xyz="0 0 0" rpy="0 0 0"/>
+        <parent link="base"/>
+        <child link="Floating Base"/>
+    </joint>
     <xacro:hipz prefix="right_" y_sign="1"/>
     <xacro:hipz prefix="left_" y_sign="-1"/>

File: robot-models/tello_humanoid.urdf (robot description, URDF)
Before this commit: robot tello_humanoid, 37 links, 36 joints
Links:
- added link torso, mass 2.3008
- link ground: mass 2.3008 -> None
Joints:
- removed joint ground-to-left-hip-clamp
- removed joint ground-to-left-hip-clamp-rotor
- removed joint ground-to-left-shoulder-ry
- removed joint ground-to-left-shoulder-ry-rotor
- removed joint ground-to-right-hip-clamp
- removed joint ground-to-right-hip-clamp-rotor
- removed joint ground-to-right-shoulder-ry
- removed joint ground-to-right-shoulder-ry-rotor
- added joint torso-to-ground: type floating, parent ground, child torso, origin xyz=0 0 0 rpy=0 0 0
- added joint torso-to-left-hip-clamp: type revolute, parent torso, child left-hip-clamp, origin xyz=0.0 126e-03 -87e-03 rpy=0.0 0.0 0.0, axis 0 0 1, limit lower=-10 upper=10 effort=150 velocity=100
- added joint torso-to-left-hip-clamp-rotor: type revolute, parent torso, child left-hip-clamp-rotor, origin xyz=0.0 126e-03 -26e-03 rpy=3.1415927 0.0 0.0, axis 0 0 1, limit lower=-10 upper=10 effort=150 velocity=100
- added joint torso-to-left-shoulder-ry: type revolute, parent torso, child left-shoulder-ry, origin xyz=0.01346 0.17608 0.24657 rpy=0.0 0.0 0.0, axis 0 1 0, limit lower=-10 upper=10 effort=150 velocity=100
- added joint torso-to-left-shoulder-ry-rotor: type revolute, parent torso, child left-shoulder-ry-rotor, origin xyz=0.01346 0.16 0.24657 rpy=0.0 0.0 0.0, axis 0 1 0, limit lower=-10 upper=10 effort=150 velocity=100
- added joint torso-to-right-hip-clamp: type revolute, parent torso, child right-hip-clamp, origin xyz=0.0 -126e-03 -87e-03 rpy=0.0 0.0 0.0, axis 0 0 1, limit lower=-10 upper=10 effort=150 velocity=100
- added joint torso-to-right-hip-clamp-rotor: type revolute, parent torso, child right-hip-clamp-rotor, origin xyz=0.0 -126e-03 -26e-03 rpy=0.0 0.0 0.0, axis 0 0 1, limit lower=-10 upper=10 effort=150 velocity=100
- added joint torso-to-right-shoulder-ry: type revolute, parent torso, child right-shoulder-ry, origin xyz=0.01346 -0.17608 0.24657 rpy=0.0 0.0 0.0, axis 0 1 0, limit lower=-10 upper=10 effort=150 velocity=100
- added joint torso-to-right-shoulder-ry-rotor: type revolute, parent torso, child right-shoulder-ry-rotor, origin xyz=0.01346 -0.16 0.24657 rpy=0.0 0.0 0.0, axis 0 1 0, limit lower=-10 upper=10 effort=150 velocity=100

File: robot-models/tello_humanoid.xacro (robot description, xacro)
@@ -4,9 +4,15 @@
     <xacro:property name="base" value="ground"/>
     <!-- Torso -->
-    <xacro:torso name="${base}"/>
+    <link name="${base}" />
+    <xacro:torso name="torso"/>
+    <joint name="torso-to-${base}" type="floating">
+        <origin xyz="0 0 0" rpy="0 0 0"/>
+        <parent link="${base}"/>
+        <child link="torso"/>
+    </joint>
     <!-- Left Hip Cluster -->
-    <xacro:L_dependent_hip_clamp_rotor_joint parent="${base}"/>
+    <xacro:L_dependent_hip_clamp_rotor_joint parent="torso"/>
     <xacro:hip_clamp_rotor prefix="left-"/>
-    <xacro:L_independent_hip_clamp_joint parent="${base}"/>
+    <xacro:L_independent_hip_clamp_joint parent="torso"/>
     <xacro:hip_clamp prefix="left-"/>
     <!-- Left Hip Differentials -->
@@ -29,7 +35,7 @@
     <xacro:foot prefix="left-"/>
     <!-- Right Hip Cluster -->
-    <xacro:R_dependent_hip_clamp_rotor_joint parent="${base}"/>
+    <xacro:R_dependent_hip_clamp_rotor_joint parent="torso"/>
     <xacro:hip_clamp_rotor prefix="right-"/>
-    <xacro:R_independent_hip_clamp_joint parent="${base}"/>
+    <xacro:R_independent_hip_clamp_joint parent="torso"/>
     <xacro:hip_clamp prefix="right-"/>
     <!-- Right Hip Differentials -->
@@ -52,7 +58,7 @@
     <xacro:foot prefix="right-"/>
     <!-- Left Shoulder RY -->
-    <xacro:L_independent_shoulder_ry_joint parent="${base}"/>
+    <xacro:L_independent_shoulder_ry_joint parent="torso"/>
     <xacro:left_shoulder_ry/>
-    <xacro:L_dependent_shoulder_ry_rotor_joint parent="${base}"/>
+    <xacro:L_dependent_shoulder_ry_rotor_joint parent="torso"/>
     <xacro:shoulder_ry_rotor prefix="left-"/>
     <!-- Left Shoulder RX -->
@@ -72,7 +78,7 @@
     <xacro:elbow_rotor prefix="left-"/>
     <!-- Right Shoulder RY -->
-    <xacro:R_independent_shoulder_ry_joint parent="${base}"/>
+    <xacro:R_independent_shoulder_ry_joint parent="torso"/>
     <xacro:right_shoulder_ry/>
-    <xacro:R_dependent_shoulder_ry_rotor_joint parent="${base}"/>
+    <xacro:R_dependent_shoulder_ry_rotor_joint parent="torso"/>
     <xacro:shoulder_ry_rotor prefix="right-"/>
     <!-- Right Shoulder RX -->

File: robot-models/tello_humanoid_approximate.urdf (robot description, URDF)
Before this commit: robot tello_humanoid_approximate, 19 links, 18 joints
Links:
- removed link base
- added link ground
- added link torso, mass 2.3008
Joints:
- removed joint base-to-left-hip-clamp
- removed joint base-to-left-shoulder-ry
- removed joint base-to-right-hip-clamp
- removed joint base-to-right-shoulder-ry
- added joint torso-to-ground: type floating, parent ground, child torso, origin xyz=0 0 0 rpy=0 0 0
- added joint torso-to-left-hip-clamp: type revolute, parent torso, child left-hip-clamp, origin xyz=0.0 126e-03 -87e-03 rpy=0.0 0.0 0.0, axis 0 0 1, limit lower=-10 upper=10 effort=150 velocity=100
- added joint torso-to-left-shoulder-ry: type revolute, parent torso, child left-shoulder-ry, origin xyz=0.01346 0.17608 0.24657 rpy=0.0 0.0 0.0, axis 0 1 0, limit lower=-10 upper=10 effort=150 velocity=100
- added joint torso-to-right-hip-clamp: type revolute, parent torso, child right-hip-clamp, origin xyz=0.0 -126e-03 -87e-03 rpy=0.0 0.0 0.0, axis 0 0 1, limit lower=-10 upper=10 effort=150 velocity=100
- added joint torso-to-right-shoulder-ry: type revolute, parent torso, child right-shoulder-ry, origin xyz=0.01346 -0.17608 0.24657 rpy=0.0 0.0 0.0, axis 0 1 0, limit lower=-10 upper=10 effort=150 velocity=100

File: robot-models/tello_humanoid_approximate.xacro (robot description, xacro)
@@ -2,9 +2,15 @@
 <robot name="tello_humanoid_approximate" xmlns:xacro="http://ros.org/wiki/xacro">
     <xacro:include filename="tello_properties.xacro"/>
-    <xacro:property name="base" value="base"/>
+    <xacro:property name="base" value="ground"/>
     <!-- Torso -->
-    <xacro:torso name="${base}"/>
+    <link name="${base}" />
+    <xacro:torso name="torso"/>
+    <joint name="torso-to-${base}" type="floating">
+        <origin xyz="0 0 0" rpy="0 0 0"/>
+        <parent link="${base}"/>
+        <child link="torso"/>
+    </joint>
     <!-- Left Hip Clamp -->
-    <xacro:L_independent_hip_clamp_joint parent="${base}"/>
+    <xacro:L_independent_hip_clamp_joint parent="torso"/>
     <xacro:hip_clamp prefix="left-"/>
     <!-- Left Gimbal, Thigh -->
@@ -19,5 +25,5 @@
     <xacro:foot prefix="left-"/>
     <!-- Right Hip Clamp -->
-    <xacro:R_independent_hip_clamp_joint parent="${base}"/>
+    <xacro:R_independent_hip_clamp_joint parent="torso"/>
     <xacro:hip_clamp prefix="right-"/>
     <!-- Right Gimbal, Thigh -->
@@ -32,5 +38,5 @@
     <xacro:foot prefix="right-"/>
     <!-- Left Shoulder RY -->
-    <xacro:L_independent_shoulder_ry_joint parent="${base}"/>
+    <xacro:L_independent_shoulder_ry_joint parent="torso"/>
     <xacro:left_shoulder_ry/>
     <!-- Left Shoulder RX -->
@@ -44,5 +50,5 @@
     <xacro:left_elbow/>
     <!-- Right Shoulder RY -->
-    <xacro:R_independent_shoulder_ry_joint parent="${base}"/>
+    <xacro:R_independent_shoulder_ry_joint parent="torso"/>
     <xacro:right_shoulder_ry/>
     <!-- Right Shoulder RX -->
