Commit message: Urdf parser unit test passing

File: robot-models/mini_cheetah_base.urdf (robot description, URDF)
Before this commit: robot mini_cheetah_base, 1 links, 0 joints
Links:
- added link base
Joints:
- added joint base_to_floating_base: type floating, parent base, child Floating Base, origin xyz=0 0 0 rpy=0 0 0
