Commit message: Move urdfs to benchmarking folder

File: Benchmarking/urdfs/parallel_chains/Explicit/depth5/loop_size2.urdf (robot description, URDF)
Before this commit: robot parallel_chain, 11 links, 2 joints
Joints:
- added joint joint_1_2: type revolute, parent link_1_1, child link_1_2, origin xyz=0 1.0 0, axis 0 0 1, limit lower=-10 upper=10 effort=30 velocity=1.0
- added joint joint_1_3: type revolute, parent link_1_2, child link_1_3, origin xyz=0 1.0 0, axis 0 0 1, limit lower=-10 upper=10 effort=30 velocity=1.0
- added joint joint_1_4: type revolute, parent link_1_3, child link_1_4, origin xyz=0 1.0 0, axis 0 0 1, limit lower=-10 upper=10 effort=30 velocity=1.0
- added joint joint_1_5: type revolute, parent link_1_4, child link_1_5, origin xyz=0 1.0 0, axis 0 0 1, limit lower=-10 upper=10 effort=30 velocity=1.0
- added joint joint_2_2: type revolute, parent link_2_1, child link_2_2, origin xyz=0 1.0 0, axis 0 0 1, limit lower=-10 upper=10 effort=30 velocity=1.0
- added joint joint_2_3: type revolute, parent link_2_2, child link_2_3, origin xyz=0 1.0 0, axis 0 0 1, limit lower=-10 upper=10 effort=30 velocity=1.0
- added joint joint_2_4: type revolute, parent link_2_3, child link_2_4, origin xyz=0 1.0 0, axis 0 0 1, limit lower=-10 upper=10 effort=30 velocity=1.0
- added joint joint_2_5: type revolute, parent link_2_4, child link_2_5, origin xyz=0 1.0 0, axis 0 0 1, limit lower=-10 upper=10 effort=30 velocity=1.0
- joint joint_2_1: origin xyz=0.25 0 0 -> xyz=0 0 0
