Commit message: Approx and rotor benchmarks working

File: Benchmarking/urdfs/four_bar_properties.xacro (robot description, xacro)
@@ -90,5 +90,5 @@
     </xacro:macro>
     <xacro:macro name="constraint" params="name predecessor successor">
-        <constraint name="${name}" type="position">
+        <loop name="${name}" type="revolute">
             <predecessor link="${predecessor}">
                 <origin xyz="0.5 0.0 0.0"/>
@@ -97,5 +97,6 @@
                 <origin xyz="1.0 0.0 0.0"/>
             </successor>
-        </constraint>
+            <axis xyz="0 0 1"/>
+        </loop>
     </xacro:macro>
     <xacro:macro name="root_branch" params="branch_count">

File: Benchmarking/urdfs/revolute_rotor_properties.xacro (robot description, xacro)
@@ -46,9 +46,9 @@
     </xacro:macro>
     <xacro:macro name="transmission" params="name predecessor successor">
-        <constraint name="${name}" type="rolling">
+        <coupling name="${name}">
             <predecessor link="${predecessor}"/>
             <successor link="${successor}"/>
             <ratio value="6.0"/>
-        </constraint>
+        </coupling>
     </xacro:macro>
     <xacro:macro name="root_branch" params="branch_count">

File: robot-models/mini_cheetah_properties.xacro (robot description, xacro)
@@ -44,6 +44,4 @@
         </link>
         <coupling name="${prefix}_abad_tranmission">
-            <predecessor link="${prefix}_abad_link"/>
-            <successor link="${prefix}_abad_rotor"/>
             <predecessor link="${prefix}_abad_link"/>
             <successor link="${prefix}_abad_rotor"/>
