Commit message: Make branch and depth robots floating base

File: Benchmarking/urdfs/four_bar_branch.xacro (robot description, xacro)
@@ -22,5 +22,18 @@
         </xacro:if>
     </xacro:macro>
-    <link name="base"/>
+    <link name="ground"/>
+    <link name="Floating Base">
+        <inertial>
+            <mass value="5.0"/>
+            <origin xyz="0. 0. 0."/>
+            <inertia ixx="0.1" ixy="0."  ixz="0."
+                     iyy="0.1" iyz="0." izz="0.1"/>
+        </inertial>
+    </link>
+    <joint name="world_to_base" type="floating">
+        <origin xyz="0 0 0" rpy="0 0 0"/>
+        <parent link="ground"/>
+        <child link="Floating Base"/>
+    </joint>
     <xacro:root_branch branch_count="${branch_count}"/>
     <xacro:build_four_bar_series_chain_at_each_branch branch_count="${branch_count}"

File: Benchmarking/urdfs/four_bar_properties.xacro (robot description, xacro)
@@ -106,8 +106,8 @@
             <xacro:L3 name="link_${(branch_count - 1) * 3 + 3}"/>
             <xacro:J1 name="base_to_link_${(branch_count - 1) * 3 + 1}"
-                      parent_link="base"
+                      parent_link="Floating Base"
                       child_link="link_${(branch_count - 1) * 3 + 1}"/>
             <xacro:J2 name="base_to_link_${(branch_count - 1) * 3 + 2}"
-                      parent_link="base"
+                      parent_link="Floating Base"
                       child_link="link_${(branch_count - 1 ) * 3 + 2}"/>
             <xacro:J3 name="link_${(branch_count - 1) * 3 + 2}_to_link_${(branch_count - 1) * 3 + 3}"

File: Benchmarking/urdfs/revolute_rotor_branch.xacro (robot description, xacro)
@@ -20,5 +20,18 @@
         </xacro:if>
     </xacro:macro>
-    <link name="base"/>
+    <link name="ground"/>
+    <link name="Floating Base">
+        <inertial>
+            <mass value="5.0"/>
+            <origin xyz="0. 0. 0."/>
+            <inertia ixx="0.1" ixy="0."  ixz="0."
+                     iyy="0.1" iyz="0." izz="0.1"/>
+        </inertial>
+    </link>
+    <joint name="world_to_base" type="floating">
+        <origin xyz="0 0 0" rpy="0 0 0"/>
+        <parent link="ground"/>
+        <child link="Floating Base"/>
+    </joint>
     <xacro:root_branch branch_count="${branch_count}"/>
     <xacro:build_series_chain_at_each_branch branch_count="${branch_count}"

File: Benchmarking/urdfs/revolute_rotor_pair_branch.xacro (robot description, xacro)
@@ -21,5 +21,18 @@
         </xacro:if>
     </xacro:macro>
-    <link name="base"/>
+    <link name="ground"/>
+    <link name="Floating Base">
+        <inertial>
+            <mass value="5.0"/>
+            <origin xyz="0. 0. 0."/>
+            <inertia ixx="0.1" ixy="0."  ixz="0."
+                     iyy="0.1" iyz="0." izz="0.1"/>
+        </inertial>
+    </link>
+    <joint name="world_to_base" type="floating">
+        <origin xyz="0 0 0" rpy="0 0 0"/>
+        <parent link="ground"/>
+        <child link="Floating Base"/>
+    </joint>
     <xacro:revolute_rotor_pair_root_branch branch_count="${branch_count}"/>
     <xacro:build_revolute_rotor_pair_series_chain_at_each_branch branch_count="${branch_count}"

File: Benchmarking/urdfs/revolute_rotor_pair_properties.xacro (robot description, xacro)
@@ -29,9 +29,9 @@
         <xacro:if value="${branch_count}">
             <xacro:independent_joint name="base_to_link_${branch_count * 2 - 1}"
-                parent="base"
+                parent="Floating Base"
                 child="link_${branch_count * 2 - 1}"/>
             <xacro:link name="link_${branch_count * 2 - 1}"/>
             <xacro:dependent_joint name="base_to_rotor_${branch_count * 2 - 1}"
-                parent="base"
+                parent="Floating Base"
                 child="rotor_${branch_count * 2 - 1}"/>
             <xacro:rotor name="rotor_${branch_count * 2 - 1}"/>
@@ -44,5 +44,5 @@
             <xacro:link name="link_${branch_count * 2}"/>
             <xacro:dependent_joint name="base_to_rotor_${branch_count * 2}"
-                parent="base" child="rotor_${branch_count * 2}"/>
+                parent="Floating Base" child="rotor_${branch_count * 2}"/>
             <xacro:rotor name="rotor_${branch_count * 2}"/>
             <xacro:transmission name="transmission_${branch_count * 2}"

File: Benchmarking/urdfs/revolute_rotor_properties.xacro (robot description, xacro)
@@ -55,8 +55,10 @@
         <xacro:if value="${branch_count}">
             <xacro:independent_joint name="base_to_link_${branch_count}"
-                                     parent="base" child="link_${branch_count}"/>
+                                     parent="Floating Base"
+                                     child="link_${branch_count}"/>
             <xacro:link name="link_${branch_count}"/>
             <xacro:dependent_joint name="base_to_rotor_${branch_count}"
-                                   parent="base" child="rotor_${branch_count}"/>
+                                   parent="Floating Base"
+                                   child="rotor_${branch_count}"/>
             <xacro:rotor name="rotor_${branch_count}"/>
             <xacro:transmission name="transmission_${branch_count}"

File: Benchmarking/urdfs/variable_four_bar_urdf/four_bar_branch_1_1.urdf (robot description, URDF)
Before this commit: robot variable_four_bar_branch, 4 links, 3 joints
Links:
- removed link base
- added link Floating Base, mass 5.0
- added link ground
Joints:
- added joint world_to_base: type floating, parent ground, child Floating Base, origin xyz=0 0 0 rpy=0 0 0
- joint base_to_link_1: parent base -> Floating Base
- joint base_to_link_2: parent base -> Floating Base

File: Benchmarking/urdfs/variable_four_bar_urdf/four_bar_branch_1_10.urdf (robot description, URDF)
Before this commit: robot variable_four_bar_branch, 31 links, 30 joints
Links:
- removed link base
- added link Floating Base, mass 5.0
- added link ground
Joints:
- added joint world_to_base: type floating, parent ground, child Floating Base, origin xyz=0 0 0 rpy=0 0 0
- joint base_to_link_1: parent base -> Floating Base
- joint base_to_link_2: parent base -> Floating Base

File: Benchmarking/urdfs/variable_four_bar_urdf/four_bar_branch_1_2.urdf (robot description, URDF)
Before this commit: robot variable_four_bar_branch, 7 links, 6 joints
Links:
- removed link base
- added link Floating Base, mass 5.0
- added link ground
Joints:
- added joint world_to_base: type floating, parent ground, child Floating Base, origin xyz=0 0 0 rpy=0 0 0
- joint base_to_link_1: parent base -> Floating Base
- joint base_to_link_2: parent base -> Floating Base

File: Benchmarking/urdfs/variable_four_bar_urdf/four_bar_branch_1_3.urdf (robot description, URDF)
Before this commit: robot variable_four_bar_branch, 10 links, 9 joints
Links:
- removed link base
- added link Floating Base, mass 5.0
- added link ground
Joints:
- added joint world_to_base: type floating, parent ground, child Floating Base, origin xyz=0 0 0 rpy=0 0 0
- joint base_to_link_1: parent base -> Floating Base
- joint base_to_link_2: parent base -> Floating Base

File: Benchmarking/urdfs/variable_four_bar_urdf/four_bar_branch_1_4.urdf (robot description, URDF)
Before this commit: robot variable_four_bar_branch, 13 links, 12 joints
Links:
- removed link base
- added link Floating Base, mass 5.0
- added link ground
Joints:
- added joint world_to_base: type floating, parent ground, child Floating Base, origin xyz=0 0 0 rpy=0 0 0
- joint base_to_link_1: parent base -> Floating Base
- joint base_to_link_2: parent base -> Floating Base

File: Benchmarking/urdfs/variable_four_bar_urdf/four_bar_branch_1_5.urdf (robot description, URDF)
Before this commit: robot variable_four_bar_branch, 16 links, 15 joints
Links:
- removed link base
- added link Floating Base, mass 5.0
- added link ground
Joints:
- added joint world_to_base: type floating, parent ground, child Floating Base, origin xyz=0 0 0 rpy=0 0 0
- joint base_to_link_1: parent base -> Floating Base
- joint base_to_link_2: parent base -> Floating Base

File: Benchmarking/urdfs/variable_four_bar_urdf/four_bar_branch_1_6.urdf (robot description, URDF)
Before this commit: robot variable_four_bar_branch, 19 links, 18 joints
Links:
- removed link base
- added link Floating Base, mass 5.0
- added link ground
Joints:
- added joint world_to_base: type floating, parent ground, child Floating Base, origin xyz=0 0 0 rpy=0 0 0
- joint base_to_link_1: parent base -> Floating Base
- joint base_to_link_2: parent base -> Floating Base

File: Benchmarking/urdfs/variable_four_bar_urdf/four_bar_branch_1_7.urdf (robot description, URDF)
Before this commit: robot variable_four_bar_branch, 22 links, 21 joints
Links:
- removed link base
- added link Floating Base, mass 5.0
- added link ground
Joints:
- added joint world_to_base: type floating, parent ground, child Floating Base, origin xyz=0 0 0 rpy=0 0 0
- joint base_to_link_1: parent base -> Floating Base
- joint base_to_link_2: parent base -> Floating Base

File: Benchmarking/urdfs/variable_four_bar_urdf/four_bar_branch_1_8.urdf (robot description, URDF)
Before this commit: robot variable_four_bar_branch, 25 links, 24 joints
Links:
- removed link base
- added link Floating Base, mass 5.0
- added link ground
Joints:
- added joint world_to_base: type floating, parent ground, child Floating Base, origin xyz=0 0 0 rpy=0 0 0
- joint base_to_link_1: parent base -> Floating Base
- joint base_to_link_2: parent base -> Floating Base

File: Benchmarking/urdfs/variable_four_bar_urdf/four_bar_branch_1_9.urdf (robot description, URDF)
Before this commit: robot variable_four_bar_branch, 28 links, 27 joints
Links:
- removed link base
- added link Floating Base, mass 5.0
- added link ground
Joints:
- added joint world_to_base: type floating, parent ground, child Floating Base, origin xyz=0 0 0 rpy=0 0 0
- joint base_to_link_1: parent base -> Floating Base
- joint base_to_link_2: parent base -> Floating Base

File: Benchmarking/urdfs/variable_four_bar_urdf/four_bar_branch_2_1.urdf (robot description, URDF)
Before this commit: robot variable_four_bar_branch, 7 links, 6 joints
Links:
- removed link base
- added link Floating Base, mass 5.0
- added link ground
Joints:
- added joint world_to_base: type floating, parent ground, child Floating Base, origin xyz=0 0 0 rpy=0 0 0
- joint base_to_link_1: parent base -> Floating Base
- joint base_to_link_2: parent base -> Floating Base
- joint base_to_link_4: parent base -> Floating Base
- joint base_to_link_5: parent base -> Floating Base

File: Benchmarking/urdfs/variable_four_bar_urdf/four_bar_branch_2_10.urdf (robot description, URDF)
Before this commit: robot variable_four_bar_branch, 61 links, 60 joints
Links:
- removed link base
- added link Floating Base, mass 5.0
- added link ground
Joints:
- added joint world_to_base: type floating, parent ground, child Floating Base, origin xyz=0 0 0 rpy=0 0 0
- joint base_to_link_1: parent base -> Floating Base
- joint base_to_link_2: parent base -> Floating Base
- joint base_to_link_4: parent base -> Floating Base
- joint base_to_link_5: parent base -> Floating Base

File: Benchmarking/urdfs/variable_four_bar_urdf/four_bar_branch_2_2.urdf (robot description, URDF)
Before this commit: robot variable_four_bar_branch, 13 links, 12 joints
Links:
- removed link base
- added link Floating Base, mass 5.0
- added link ground
Joints:
- added joint world_to_base: type floating, parent ground, child Floating Base, origin xyz=0 0 0 rpy=0 0 0
- joint base_to_link_1: parent base -> Floating Base
- joint base_to_link_2: parent base -> Floating Base
- joint base_to_link_4: parent base -> Floating Base
- joint base_to_link_5: parent base -> Floating Base

File: Benchmarking/urdfs/variable_four_bar_urdf/four_bar_branch_2_3.urdf (robot description, URDF)
Before this commit: robot variable_four_bar_branch, 19 links, 18 joints
Links:
- removed link base
- added link Floating Base, mass 5.0
- added link ground
Joints:
- added joint world_to_base: type floating, parent ground, child Floating Base, origin xyz=0 0 0 rpy=0 0 0
- joint base_to_link_1: parent base -> Floating Base
- joint base_to_link_2: parent base -> Floating Base
- joint base_to_link_4: parent base -> Floating Base
- joint base_to_link_5: parent base -> Floating Base
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