Commit message: Fix bug with nca to pred and succ. Parallel chain benchmark now passing

File: Benchmarking/urdfs/parallel_chains/Implicit/implicit_parallel_chains_properties.xacro (robot description, xacro)
@@ -36,5 +36,5 @@
             <limit effort="30" velocity="1.0" lower="-10" upper="10"/>
         </joint>
-        <constraint name="position_${idx}" type="position">
+        <loop name="position_${idx}" type="revolute">
             <predecessor link="connecting_rod">
                 <origin xyz="${distance_between_chains} 0.0 0.0"/>
@@ -43,5 +43,6 @@
                 <origin xyz="0.0 ${link_length} 0.0"/>
             </successor>
-        </constraint>
+            <axis xyz="0 0 1"/>
+        </loop>
     </xacro:macro>
     <xacro:macro name="add_constrained_parallel_links_and_joints" params="idx">
